File: Hardware/Core.sch (KiCad schematic (older format))
At the start: 22 parts, among them U1 AAT1217, U3 MSP430G2553-PW28, U4 MCP6L02T

Commit message: Something changed
Parts:
- gave numbers to parts that had none: 3
- renumbered C1 to C24, C12 to C25, C12 to C26, C13 to C27, C3 to C28, C2 to C29, C14 to C30, C15 to C32, C11 to C34, L1 to L8, R6 to R10, R7 to R11, R8 to R12, R4 to R13, R5 to R8, R1 to R9, U1 to U3, U3 to U5
Connections:
- net Mod: no longer R8.1
- new net AF: R8.1
Changed lines of the file:
@@
 Sheet 4 4
 Title "Aether - Pico Tracker"
-Date "3 feb 2014"
+Date "4 feb 2014"
 Rev "1"
 Comp "Aerodyne Labs"
@@
 $EndDescr
 $Comp
-L AAT1217 U1
+L AAT1217 U3
 U 1 1 52ECD611
 P 2600 2300
-F 0 "U1" H 2600 2800 60  0000 C CNN
+F 0 "U3" H 2600 2800 60  0000 C CNN
 F 1 "AAT1217" V 2600 2300 60  0000 C CNN
 F 2 "" H 2600 2300 60  0000 C CNN
@@
 $EndComp
 $Comp
-L L L1
+L L L8
 U 1 1 52ECD617
 P 2600 1500
-F 0 "L1" H 2600 1400 60  0000 C CNN
+F 0 "L8" H 2600 1400 60  0000 C CNN
 F 1 "4.7uH" H 2600 1550 60  0000 C CNN
 F 2 "INDC3225-N" H 2600 1500 60  0001 C CNN
@@
 $EndComp
 $Comp
-L R R1
+L R R9
 U 1 1 52ECD628
 P 2000 2250
-F 0 "R1" H 2000 2350 50  0000 C CNN
+F 0 "R9" H 2000 2350 50  0000 C CNN
 F 1 "10k" H 2000 2250 50  0000 C CNN
 F 2 "RESC1608-N" H 2000 2250 60  0001 C CNN
@@
 $EndComp
 $Comp
-L C C1
+L C C24
 U 1 1 52ECD632
 P 1600 2250
-F 0 "C1" H 1650 2400 60  0000 L CNN
+F 0 "C24" H 1650 2400 60  0000 L CNN
 F 1 "4.7uF" H 1650 2100 60  0000 L CNN
 F 2 "CAPC2012-N" H 1600 2250 60  0001 C CNN
@@
 $EndComp
 $Comp
-L +BATT #PWR?
+L +BATT #PWR041
 U 1 1 52ECD638
 P 1600 1800
-F 0 "#PWR?" H 1600 1750 20  0001 C CNN
+F 0 "#PWR041" H 1600 1750 20  0001 C CNN
 F 1 "+BATT" H 1600 1900 30  0000 C CNN
 F 2 "" H 1600 1800 60  0000 C CNN
@@
 $EndComp
 $Comp
-L GND #PWR?
+L GND #PWR042
 U 1 1 52ECD64A
 P 3600 2700
-F 0 "#PWR?" H 3600 2700 30  0001 C CNN
+F 0 "#PWR042" H 3600 2700 30  0001 C CNN
 F 1 "GND" H 3600 2630 30  0001 C CNN
 F 2 "" H 3600 2700 60  0000 C CNN
@@
 $EndComp
 $Comp
-L GND #PWR?
+L GND #PWR043
 U 1 1 52ECD650
 P 1600 2600
-F 0 "#PWR?" H 1600 2600 30  0001 C CNN
+F 0 "#PWR043" H 1600 2600 30  0001 C CNN
 F 1 "GND" H 1600 2530 30  0001 C CNN
 F 2 "" H 1600 2600 60  0000 C CNN
@@
 $EndComp
 $Comp
-L GND #PWR?
+L GND #PWR044
 U 1 1 52ECD656
 P 2000 2800
-F 0 "#PWR?" H 2000 2800 30  0001 C CNN
+F 0 "#PWR044" H 2000 2800 30  0001 C CNN
 F 1 "GND" H 2000 2730 30  0001 C CNN
 F 2 "" H 2000 2800 60  0000 C CNN
@@
 $EndComp
 $Comp
-L +3.3V #PWR?
+L +3.3V #PWR045
 U 1 1 52ECD663
 P 3600 1800
-F 0 "#PWR?" H 3600 1760 30  0001 C CNN
+F 0 "#PWR045" H 3600 1760 30  0001 C CNN
 F 1 "+3.3V" H 3600 1910 30  0000 C CNN
 F 2 "" H 3600 1800 60  0000 C CNN
@@
 $EndComp
 $Comp
-L GND #PWR?
+L GND #PWR046
 U 1 1 52ECE5C9
 P 8800 4000
-F 0 "#PWR?" H 8800 4000 30  0001 C CNN
+F 0 "#PWR046" H 8800 4000 30  0001 C CNN
 F 1 "GND" H 8800 3930 30  0001 C CNN
 F 2 "" H 8800 4000 60  0000 C CNN
@@
 $EndComp
 $Comp
-L +3.3V #PWR?
+L +3.3V #PWR047
 U 1 1 52ECE681
 P 8900 2000
-F 0 "#PWR?" H 8900 1960 30  0001 C CNN
+F 0 "#PWR047" H 8900 1960 30  0001 C CNN
 F 1 "+3.3V" H 8900 2110 30  0000 C CNN
 F 2 "" H 8900 2000 60  0000 C CNN
@@
 $EndComp
 $Comp
-L +3.3V #PWR?
+L +3.3V #PWR048
 U 1 1 52ECE6CC
 P 7200 2000
-F 0 "#PWR?" H 7200 1960 30  0001 C CNN
+F 0 "#PWR048" H 7200 1960 30  0001 C CNN
 F 1 "+3.3V" H 7200 2110 30  0000 C CNN
 F 2 "" H 7200 2000 60  0000 C CNN
@@
 $EndComp
 $Comp
-L C C11
+L C C34
 U 1 1 52ECE6FD
 P 7550 2200
-F 0 "C11" H 7600 2350 60  0000 L CNN
+F 0 "C34" H 7600 2350 60  0000 L CNN
 F 1 "0.1uF" H 7600 2050 60  0000 L CNN
 F 2 "CAPC1608-N" H 7550 2200 60  0001 C CNN
@@
 $EndComp
 $Comp
-L GND #PWR?
+L GND #PWR049
 U 1 1 52ECE742
 P 7900 2200
-F 0 "#PWR?" H 7900 2200 30  0001 C CNN
+F 0 "#PWR049" H 7900 2200 30  0001 C CNN
 F 1 "GND" H 7900 2130 30  0001 C CNN
 F 2 "" H 7900 2200 60  0000 C CNN
@@
 $EndComp
 $Comp
-L R R5
+L R R8
 U 1 1 52EDECAB
 P 1450 6200
-F 0 "R5" H 1450 6300 50  0000 C CNN
+F 0 "R8" H 1450 6300 50  0000 C CNN
 F 1 "16k" H 1450 6200 50  0000 C CNN
 F 2 "RESC1608-N" H 1450 6200 60  0001 C CNN
@@
 $EndComp
 $Comp
-L GND #PWR?
+L GND #PWR050
 U 1 1 52EDECF2
 P 3100 6500
-F 0 "#PWR?" H 3100 6500 30  0001 C CNN
+F 0 "#PWR050" H 3100 6500 30  0001 C CNN
 F 1 "GND" H 3100 6430 30  0001 C CNN
 F 2 "" H 3100 6500 60  0000 C CNN
@@
 $EndComp
 $Comp
-L GND #PWR?
+L GND #PWR051
 U 1 1 52EDED01
 P 2500 7000
-F 0 "#PWR?" H 2500 7000 30  0001 C CNN
+F 0 "#PWR051" H 2500 7000 30  0001 C CNN
 F 1 "GND" H 2500 6930 30  0001 C CNN
 F 2 "" H 2500 7000 60  0000 C CNN
@@
 $EndComp
 $Comp
-L GND #PWR?
+L GND #PWR052
 U 1 1 52EDF036
 P 5100 6800
-F 0 "#PWR?" H 5100 6800 30  0001 C CNN
+F 0 "#PWR052" H 5100 6800 30  0001 C CNN
 F 1 "GND" H 5100 6730 30  0001 C CNN
 F 2 "" H 5100 6800 60  0000 C CNN
@@
 $EndComp
 $Comp
-L GND #PWR?
+L GND #PWR053
 U 1 1 52EDF155
 P 1800 5500
-F 0 "#PWR?" H 1800 5500 30  0001 C CNN
+F 0 "#PWR053" H 1800 5500 30  0001 C CNN
 F 1 "GND" H 1800 5430 30  0001 C CNN
 F 2 "" H 1800 5500 60  0000 C CNN
@@
 Connection ~ 6300 5800
 $Comp
-L +3.3V #PWR?
+L +3.3V #PWR054
 U 1 1 52EDF302
 P 3100 5300
-F 0 "#PWR?" H 3100 5260 30  0001 C CNN
+F 0 "#PWR054" H 3100 5260 30  0001 C CNN
 F 1 "+3.3V" H 3100 5410 30  0000 C CNN
 F 2 "" H 3100 5300 60  0000 C CNN
@@
 	1800 5400 1900 5400
 Text Label 1100 6200 2    60   ~ 0
-Mod
+AF
 Wire Wire Line
 	1100 6200 1200 6200
 Text Label 6500 3800 2    60   ~ 0
-Mod
+AF
 Text HLabel 6500 3500 0    60   Output ~ 0
 GPS_Perf
 $Comp
-L CRYSTAL X?
+L CRYSTAL X2
 U 1 1 52EF2F5E
 P 5150 1700
-F 0 "X?" H 5150 1850 60  0000 C CNN
+F 0 "X2" H 5150 1850 60  0000 C CNN
 F 1 "CRYSTAL" H 5150 1550 60  0000 C CNN
 F 2 "~" H 5150 1700 60  0000 C CNN
@@
 $EndComp
 $Comp
-L C C?
+L C C33
 U 1 1 52EF2F6D
 P 5500 2050
-F 0 "C?" H 5550 2200 60  0000 L CNN
+F 0 "C33" H 5550 2200 60  0000 L CNN
 F 1 "C" H 5550 1900 60  0000 L CNN
 F 2 "~" H 5500 2050 60  0000 C CNN
@@
 $EndComp
 $Comp
-L C C?
+L C C31
 U 1 1 52EF2F88
 P 4800 2050
-F 0 "C?" H 4850 2200 60  0000 L CNN
+F 0 "C31" H 4850 2200 60  0000 L CNN
 F 1 "C" H 4850 1900 60  0000 L CNN
 F 2 "~" H 4800 2050 60  0000 C CNN
@@
 Connection ~ 4800 1700
 $Comp
-L GND #PWR?
+L GND #PWR055
 U 1 1 52EF30D2
 P 5500 2400
-F 0 "#PWR?" H 5500 2400 30  0001 C CNN
+F 0 "#PWR055" H 5500 2400 30  0001 C CNN
 F 1 "GND" H 5500 2330 30  0001 C CNN
 F 2 "" H 5500 2400 60  0000 C CNN
@@
 $EndComp
 $Comp
-L GND #PWR?
+L GND #PWR056
 U 1 1 52EF30E1
 P 4800 2400
-F 0 "#PWR?" H 4800 2400 30  0001 C CNN
+F 0 "#PWR056" H 4800 2400 30  0001 C CNN
 F 1 "GND" H 4800 2330 30  0001 C CNN
 F 2 "" H 4800 2400 60  0000 C CNN
@@
 	8700 2800 9000 2800
 $Comp
-L C C3
+L C C28
 U 1 1 52EF39D3
 P 3200 2350
-F 0 "C3" H 3250 2500 60  0000 L CNN
+F 0 "C28" H 3250 2500 60  0000 L CNN
 F 1 "DNP" H 3250 2200 60  0000 L CNN
 F 2 "CAPC1608-N" H 3200 2350 60  0001 C CNN
@@
 	3200 2700 3100 2700
 $Comp
-L C C2
+L C C29
 U 1 1 52EF6065
 P 3600 2350
-F 0 "C2" H 3650 2500 60  0000 L CNN
+F 0 "C29" H 3650 2500 60  0000 L CNN
 F 1 "4.7uF" H 3650 2200 60  0000 L CNN
 F 2 "CAPC2012-N" H 3600 2350 60  0001 C CNN
@@
 	9000 3200 8700 3200
 $Comp
-L R R4
+L R R13
 U 1 1 52EF83E3
 P 8900 2350
-F 0 "R4" H 8900 2450 50  0000 C CNN
+F 0 "R13" H 8900 2450 50  0000 C CNN
 F 1 "10k" H 8900 2350 50  0000 C CNN
 F 2 "RESC1608-N" H 8900 2350 60  0001 C CNN
@@
 	7200 2200 7300 2200
 $Comp
-L MSP430G2553-PW28 U3
+L MSP430G2553-PW28 U5
 U 1 1 52EFA4DC
 P 8000 3250
-F 0 "U3" H 8000 4000 60  0000 C CNN
+F 0 "U5" H 8000 4000 60  0000 C CNN
 F 1 "MSP430G2553-PW28" H 8000 2500 60  0000 C CNN
 F 2 "" H 8000 2400 60  0000 C CNN
@@
 Stat
 $Comp
-L +BATT #PWR?
+L +BATT #PWR057
 U 1 1 52EFA84C
 P 7000 2200
-F 0 "#PWR?" H 7000 2150 20  0001 C CNN
+F 0 "#PWR057" H 7000 2150 20  0001 C CNN
 F 1 "+BATT" H 7000 2300 30  0000 C CNN
 F 2 "" H 7000 2200 60  0000 C CNN
@@
 	7000 2700 7300 2700
 $Comp
-L C C12
+L C C25
 U 1 1 52F025C5
 P 1800 6550
-F 0 "C12" H 1850 6700 60  0000 L CNN
+F 0 "C25" H 1850 6700 60  0000 L CNN
 F 1 "1000pF" H 1850 6400 60  0000 L CNN
 F 2 "CAPC1608-N" H 1800 6550 60  0001 C CNN
@@
 $EndComp
 $Comp
-L C C12
+L C C26
 U 1 1 52F02988
 P 2150 5400
-F 0 "C12" H 2200 5550 60  0000 L CNN
+F 0 "C26" H 2200 5550 60  0000 L CNN
 F 1 "0.1uF" H 2200 5250 60  0000 L CNN
 F 2 "CAPC1608-N" H 2150 5400 60  0001 C CNN
@@
 	5100 5300 6300 5300
 $Comp
-L R R6
+L R R10
 U 1 1 52F02A80
 P 2150 6200
-F 0 "R6" H 2150 6300 50  0000 C CNN
+F 0 "R10" H 2150 6300 50  0000 C CNN
 F 1 "16k" H 2150 6200 50  0000 C CNN
 F 2 "RESC1608-N" H 2150 6200 60  0001 C CNN
@@
 $EndComp
 $Comp
-L R R7
+L R R11
 U 1 1 52F02A8B
 P 4050 6000
-F 0 "R7" H 4050 6100 50  0000 C CNN
+F 0 "R11" H 4050 6100 50  0000 C CNN
 F 1 "16k" H 4050 6000 50  0000 C CNN
 F 2 "RESC1608-N" H 4050 6000 60  0001 C CNN
@@
 $EndComp
 $Comp
-L R R8
+L R R12
 U 1 1 52F02A96
 P 4750 6000
-F 0 "R8" H 4750 6100 50  0000 C CNN
+F 0 "R12" H 4750 6100 50  0000 C CNN
 F 1 "16k" H 4750 6000 50  0000 C CNN
 F 2 "RESC1608-N" H 4750 6000 60  0001 C CNN
@@
 $EndComp
 $Comp
-L C C13
+L C C27
 U 1 1 52F02B45
 P 2500 6550
-F 0 "C13" H 2550 6700 60  0000 L CNN
+F 0 "C27" H 2550 6700 60  0000 L CNN
 F 1 "1000pF" H 2550 6400 60  0000 L CNN
 F 2 "CAPC1608-N" H 2500 6550 60  0001 C CNN
@@
 $EndComp
 $Comp
-L C C14
+L C C30
 U 1 1 52F02B50
 P 4400 6350
-F 0 "C14" H 4450 6500 60  0000 L CNN
+F 0 "C30" H 4450 6500 60  0000 L CNN
 F 1 "1000pF" H 4450 6200 60  0000 L CNN
 F 2 "CAPC1608-N" H 4400 6350 60  0001 C CNN
@@
 $EndComp
 $Comp
-L C C15
+L C C32
 U 1 1 52F02B5B
 P 5100 6350
-F 0 "C15" H 5150 6500 60  0000 L CNN
+F 0 "C32" H 5150 6500 60  0000 L CNN
 F 1 "1000pF" H 5150 6200 60  0000 L CNN
 F 2 "CAPC1608-N" H 5100 6350 60  0001 C CNN
