File: Hardware/Core.sch (KiCad schematic (older format))
At the start: 23 parts, among them U3 AAT1217, U4 MCP6L02T, U5 MSP430G2553-PW28, X2 8MHz

Commit message: Voltage regulator components
Parts:
- C28: footprint CAPC1608-N -> CAPC1005-N
- R9: footprint RESC1608-N -> RESC1005-N; Distributor Part No 311-10KGRCT-ND -> RMCF0402JT10K0CT-ND; MFR Name Yageo -> Stackpole; MFR Part No RC0603JR-0710KL -> RMCF0402JT10K0; Power 0.1W -> 1/16W
Changed lines of the file:
@@
 F 0 "R9" H 2000 2350 50  0000 C CNN
 F 1 "10k" H 2000 2250 50  0000 C CNN
-F 2 "RESC1608-N" H 2000 2250 60  0001 C CNN
+F 2 "RESC1005-N" H 2000 2250 60  0001 C CNN
 F 3 "~" H 2000 2250 60  0000 C CNN
-F 4 "Yageo" H 2000 2250 60  0001 C CNN "MFR Name"
-F 5 "RC0603JR-0710KL" H 2000 2250 60  0001 C CNN "MFR Part No"
-F 6 "311-10KGRCT-ND" H 2000 2250 60  0001 C CNN "Distributor Part No"
-F 7 "0.1W" H 2000 2150 50  0001 C CNN "Power"
+F 4 "Stackpole" H 2000 2250 60  0001 C CNN "MFR Name"
+F 5 "RMCF0402JT10K0" H 2000 2250 60  0001 C CNN "MFR Part No"
+F 6 "RMCF0402JT10K0CT-ND" H 2000 2250 60  0001 C CNN "Distributor Part No"
+F 7 "1/16W" H 2000 2150 50  0001 C CNN "Power"
 F 8 "5%" H 2000 2050 50  0001 C CNN "Tolerance"
 	1    2000 2250
@@
 $EndComp
 $Comp
-L C C24
-U 1 1 52ECD632
-P 1600 2250
-F 0 "C24" H 1650 2400 60  0000 L CNN
-F 1 "4.7uF" H 1650 2100 60  0000 L CNN
-F 2 "CAPC2012-N" H 1600 2250 60  0001 C CNN
-F 3 "~" H 1600 2250 60  0000 C CNN
-F 4 "Samsung" H 1600 2250 60  0001 C CNN "MFR Name"
-F 5 "CL21A475KOFNNNE" H 1600 2250 60  0001 C CNN "MFR Part No"
-F 6 "1276-1065-1-ND" H 1600 2250 60  0001 C CNN "Distributor Part No"
-F 7 "16V" H 1550 2100 60  0001 R CNN "Voltage"
-F 8 "X5R" H 1550 2400 60  0001 R CNN "Dielectric"
-	1    1600 2250
-	-1   0    0    -1
-$EndComp
-$Comp
-L +BATT #PWR048
+L +BATT #PWR050
 U 1 1 52ECD638
 P 1600 1800
-F 0 "#PWR048" H 1600 1750 20  0001 C CNN
+F 0 "#PWR050" H 1600 1750 20  0001 C CNN
 F 1 "+BATT" H 1600 1900 30  0000 C CNN
 F 2 "" H 1600 1800 60  0000 C CNN
@@
 $EndComp
 $Comp
-L GND #PWR049
+L GND #PWR051
 U 1 1 52ECD64A
 P 3600 2700
-F 0 "#PWR049" H 3600 2700 30  0001 C CNN
+F 0 "#PWR051" H 3600 2700 30  0001 C CNN
 F 1 "GND" H 3600 2630 30  0001 C CNN
 F 2 "" H 3600 2700 60  0000 C CNN
@@
 $EndComp
 $Comp
-L GND #PWR050
+L GND #PWR052
 U 1 1 52ECD650
 P 1600 2600
-F 0 "#PWR050" H 1600 2600 30  0001 C CNN
+F 0 "#PWR052" H 1600 2600 30  0001 C CNN
 F 1 "GND" H 1600 2530 30  0001 C CNN
 F 2 "" H 1600 2600 60  0000 C CNN
@@
 $EndComp
 $Comp
-L GND #PWR051
+L GND #PWR053
 U 1 1 52ECD656
 P 2000 2800
-F 0 "#PWR051" H 2000 2800 30  0001 C CNN
+F 0 "#PWR053" H 2000 2800 30  0001 C CNN
 F 1 "GND" H 2000 2730 30  0001 C CNN
 F 2 "" H 2000 2800 60  0000 C CNN
@@
 $EndComp
 $Comp
-L +3.3V #PWR052
+L +3.3V #PWR054
 U 1 1 52ECD663
 P 3600 1800
-F 0 "#PWR052" H 3600 1760 30  0001 C CNN
+F 0 "#PWR054" H 3600 1760 30  0001 C CNN
 F 1 "+3.3V" H 3600 1910 30  0000 C CNN
 F 2 "" H 3600 1800 60  0000 C CNN
@@
 $EndComp
 $Comp
-L GND #PWR053
+L GND #PWR055
 U 1 1 52ECE5C9
 P 8800 4000
-F 0 "#PWR053" H 8800 4000 30  0001 C CNN
+F 0 "#PWR055" H 8800 4000 30  0001 C CNN
 F 1 "GND" H 8800 3930 30  0001 C CNN
 F 2 "" H 8800 4000 60  0000 C CNN
@@
 $EndComp
 $Comp
-L +3.3V #PWR054
+L +3.3V #PWR056
 U 1 1 52ECE681
 P 8900 2000
-F 0 "#PWR054" H 8900 1960 30  0001 C CNN
+F 0 "#PWR056" H 8900 1960 30  0001 C CNN
 F 1 "+3.3V" H 8900 2110 30  0000 C CNN
 F 2 "" H 8900 2000 60  0000 C CNN
@@
 $EndComp
 $Comp
-L +3.3V #PWR055
+L +3.3V #PWR057
 U 1 1 52ECE6CC
 P 7200 2000
-F 0 "#PWR055" H 7200 1960 30  0001 C CNN
+F 0 "#PWR057" H 7200 1960 30  0001 C CNN
 F 1 "+3.3V" H 7200 2110 30  0000 C CNN
 F 2 "" H 7200 2000 60  0000 C CNN
@@
 $EndComp
 $Comp
-L GND #PWR056
+L GND #PWR058
 U 1 1 52ECE742
 P 7900 2200
-F 0 "#PWR056" H 7900 2200 30  0001 C CNN
+F 0 "#PWR058" H 7900 2200 30  0001 C CNN
 F 1 "GND" H 7900 2130 30  0001 C CNN
 F 2 "" H 7900 2200 60  0000 C CNN
@@
 $EndComp
 $Comp
-L GND #PWR057
+L GND #PWR059
 U 1 1 52EDECF2
 P 3100 6500
-F 0 "#PWR057" H 3100 6500 30  0001 C CNN
+F 0 "#PWR059" H 3100 6500 30  0001 C CNN
 F 1 "GND" H 3100 6430 30  0001 C CNN
 F 2 "" H 3100 6500 60  0000 C CNN
@@
 $EndComp
 $Comp
-L GND #PWR058
+L GND #PWR060
 U 1 1 52EDED01
 P 2500 7000
-F 0 "#PWR058" H 2500 7000 30  0001 C CNN
+F 0 "#PWR060" H 2500 7000 30  0001 C CNN
 F 1 "GND" H 2500 6930 30  0001 C CNN
 F 2 "" H 2500 7000 60  0000 C CNN
@@
 $EndComp
 $Comp
-L GND #PWR059
+L GND #PWR061
 U 1 1 52EDF036
 P 5100 6800
-F 0 "#PWR059" H 5100 6800 30  0001 C CNN
+F 0 "#PWR061" H 5100 6800 30  0001 C CNN
 F 1 "GND" H 5100 6730 30  0001 C CNN
 F 2 "" H 5100 6800 60  0000 C CNN
@@
 $EndComp
 $Comp
-L GND #PWR060
+L GND #PWR062
 U 1 1 52EDF155
 P 1800 5500
-F 0 "#PWR060" H 1800 5500 30  0001 C CNN
+F 0 "#PWR062" H 1800 5500 30  0001 C CNN
 F 1 "GND" H 1800 5430 30  0001 C CNN
 F 2 "" H 1800 5500 60  0000 C CNN
@@
 Connection ~ 6300 5800
 $Comp
-L +3.3V #PWR061
+L +3.3V #PWR063
 U 1 1 52EDF302
 P 3100 5300
-F 0 "#PWR061" H 3100 5260 30  0001 C CNN
+F 0 "#PWR063" H 3100 5260 30  0001 C CNN
 F 1 "+3.3V" H 3100 5410 30  0000 C CNN
 F 2 "" H 3100 5300 60  0000 C CNN
@@
 Connection ~ 4800 1700
 $Comp
-L GND #PWR062
+L GND #PWR064
 U 1 1 52EF30D2
 P 5500 2400
-F 0 "#PWR062" H 5500 2400 30  0001 C CNN
+F 0 "#PWR064" H 5500 2400 30  0001 C CNN
 F 1 "GND" H 5500 2330 30  0001 C CNN
 F 2 "" H 5500 2400 60  0000 C CNN
@@
 $EndComp
 $Comp
-L GND #PWR063
+L GND #PWR065
 U 1 1 52EF30E1
 P 4800 2400
-F 0 "#PWR063" H 4800 2400 30  0001 C CNN
+F 0 "#PWR065" H 4800 2400 30  0001 C CNN
 F 1 "GND" H 4800 2330 30  0001 C CNN
 F 2 "" H 4800 2400 60  0000 C CNN
@@
 F 0 "C28" H 3250 2500 60  0000 L CNN
 F 1 "DNP" H 3250 2200 60  0000 L CNN
-F 2 "CAPC1608-N" H 3200 2350 60  0001 C CNN
+F 2 "CAPC1005-N" H 3200 2350 60  0001 C CNN
 F 3 "~" H 3200 2350 60  0000 C CNN
 F 4 "V" H 3150 2200 60  0001 R CNN "Voltage"
@@
 Wire Wire Line
 	3200 2700 3100 2700
-$Comp
-L C C29
-U 1 1 52EF6065
-P 3600 2350
-F 0 "C29" H 3650 2500 60  0000 L CNN
-F 1 "4.7uF" H 3650 2200 60  0000 L CNN
-F 2 "CAPC2012-N" H 3600 2350 60  0001 C CNN
-F 3 "~" H 3600 2350 60  0000 C CNN
-F 4 "Samsung" H 3600 2350 60  0001 C CNN "MFR Name"
-F 5 "CL21A475KOFNNNE" H 3600 2350 60  0001 C CNN "MFR Part No"
-F 6 "1276-1065-1-ND" H 3600 2350 60  0001 C CNN "Distributor Part No"
-F 7 "16V" H 3550 2200 60  0001 R CNN "Voltage"
-F 8 "X5R" H 3550 2500 60  0001 R CNN "Dielectric"
-	1    3600 2350
-	1    0    0    -1
-$EndComp
 Text HLabel 9000 3200 2    60   Output ~ 0
 SCL
@@
 Stat
 $Comp
-L +BATT #PWR064
+L +BATT #PWR066
 U 1 1 52EFA84C
 P 7000 2200
-F 0 "#PWR064" H 7000 2150 20  0001 C CNN
+F 0 "#PWR066" H 7000 2150 20  0001 C CNN
 F 1 "+BATT" H 7000 2300 30  0000 C CNN
 F 2 "" H 7000 2200 60  0000 C CNN
@@
 	-1   0    0    1
 $EndComp
+$Comp
+L C C24
+U 1 1 52F5954D
+P 1600 2250
+F 0 "C24" H 1650 2400 60  0000 L CNN
+F 1 "4.7uF" H 1650 2100 60  0000 L CNN
+F 2 "CAPC2012-N" H 1600 2250 60  0001 C CNN
+F 3 "~" H 1600 2250 60  0000 C CNN
+F 4 "Samsung" H 1600 2250 60  0001 C CNN "MFR Name"
+F 5 "CL21A475KOFNNNE" H 1600 2250 60  0001 C CNN "MFR Part No"
+F 6 "1276-1065-1-ND" H 1600 2250 60  0001 C CNN "Distributor Part No"
+F 7 "16V" H 1550 2100 60  0001 R CNN "Voltage"
+F 8 "X5R" H 1550 2400 60  0001 R CNN "Dielectric"
+	1    1600 2250
+	-1   0    0    -1
+$EndComp
+$Comp
+L C C29
+U 1 1 52F5958E
+P 3600 2350
+F 0 "C29" H 3650 2500 60  0000 L CNN
+F 1 "4.7uF" H 3650 2200 60  0000 L CNN
+F 2 "CAPC2012-N" H 3600 2350 60  0001 C CNN
+F 3 "~" H 3600 2350 60  0000 C CNN
+F 4 "Samsung" H 3600 2350 60  0001 C CNN "MFR Name"
+F 5 "CL21A475KOFNNNE" H 3600 2350 60  0001 C CNN "MFR Part No"
+F 6 "1276-1065-1-ND" H 3600 2350 60  0001 C CNN "Distributor Part No"
+F 7 "16V" H 3550 2200 60  0001 R CNN "Voltage"
+F 8 "X5R" H 3550 2500 60  0001 R CNN "Dielectric"
+	1    3600 2350
+	1    0    0    -1
+$EndComp
 $EndSCHEMATC

Commit message: Microcontroller components
Parts:
- C31, C33: value C -> 22pF; footprint ~ -> CAPC1005-N; Dielectric D -> C0G; Distributor Part No (none) -> 311-1018-1-ND; MFR Name (none) -> Yageo; MFR Part No (none) -> CC0402JRNPO9BN220; Voltage V -> 50V
- C34: footprint CAPC1608-N -> CAPC1005-N; Distributor Part No 1276-1005-1-ND -> 1276-1001-1-ND; MFR Part No CL10B104KO8NNNC -> CL05B104KO5NNNC
- R13: footprint RESC1608-N -> RESC1005-N; Distributor Part No 311-10KGRCT-ND -> RMCF0402JT10K0CT-ND; MFR Name Yageo -> Stackpole; MFR Part No RC0603JR-0710KL -> RMCF0402JT10K0; Power 0.1W -> 1/16W
- R14: footprint ~ -> RESC1005-N; Distributor Part No (none) -> RMCF0402JT10K0CT-ND; MFR Name (none) -> Stackpole; MFR Part No (none) -> RMCF0402JT10K0; Power W -> 1/16W; Tolerance % -> 5%
- X2: footprint ~ -> XTAL-2SMD-50X32; MFR Name (none) -> Abracon; MFR Part No (none) -> ABM3-8.000MHZ-D2Y-T
Changed lines of the file:
@@
-$EndComp
-$Comp
-L C C34
-U 1 1 52ECE6FD
-P 7550 2200
-F 0 "C34" H 7600 2350 60  0000 L CNN
-F 1 "0.1uF" H 7600 2050 60  0000 L CNN
-F 2 "CAPC1608-N" H 7550 2200 60  0001 C CNN
-F 3 "~" H 7550 2200 60  0000 C CNN
-F 4 "Samsung" H 7550 2200 60  0001 C CNN "MFR Name"
-F 5 "CL10B104KO8NNNC" H 7550 2200 60  0001 C CNN "MFR Part No"
-F 6 "1276-1005-1-ND" H 7550 2200 60  0001 C CNN "Distributor Part No"
-F 7 "16V" H 7500 2050 60  0001 R CNN "Voltage"
-F 8 "X7R" H 7500 2350 60  0001 R CNN "Dielectric"
-	1    7550 2200
-	0    -1   -1   0
 $EndComp
 $Comp
@@
 Text HLabel 9000 2900 2    60   Input ~ 0
 TCK/TEST
-Text HLabel 9500 3300 2    60   Input ~ 0
+Text HLabel 9600 3300 2    60   Input ~ 0
 PGM_Det
 $Comp
@@
 F 0 "X2" H 5150 1850 60  0000 C CNN
 F 1 "8MHz" H 5150 1550 60  0000 C CNN
-F 2 "~" H 5150 1700 60  0000 C CNN
+F 2 "XTAL-2SMD-50X32" H 5150 1700 60  0001 C CNN
 F 3 "~" H 5150 1700 60  0000 C CNN
-F 4 "535-10630-1-ND" H 5150 1700 60  0001 C CNN "Distributor Part No"
+F 4 "Abracon" H 5150 1700 60  0001 C CNN "MFR Name"
+F 5 "ABM3-8.000MHZ-D2Y-T" H 5150 1700 60  0001 C CNN "MFR Part No"
+F 6 "535-10630-1-ND" H 5150 1700 60  0001 C CNN "Distributor Part No"
 	1    5150 1700
 	1    0    0    -1
-$EndComp
-$Comp
-L C C33
-U 1 1 52EF2F6D
-P 5500 2050
-F 0 "C33" H 5550 2200 60  0000 L CNN
-F 1 "C" H 5550 1900 60  0000 L CNN
-F 2 "~" H 5500 2050 60  0000 C CNN
-F 3 "~" H 5500 2050 60  0000 C CNN
-F 4 "V" H 5450 1900 60  0001 R CNN "Voltage"
-F 5 "D" H 5450 2200 60  0001 R CNN "Dielectric"
-	1    5500 2050
-	1    0    0    -1
-$EndComp
-$Comp
-L C C31
-U 1 1 52EF2F88
-P 4800 2050
-F 0 "C31" H 4850 2200 60  0000 L CNN
-F 1 "C" H 4850 1900 60  0000 L CNN
-F 2 "~" H 4800 2050 60  0000 C CNN
-F 3 "~" H 4800 2050 60  0000 C CNN
-F 4 "V" H 4750 1900 60  0001 R CNN "Voltage"
-F 5 "D" H 4750 2200 60  0001 R CNN "Dielectric"
-	1    4800 2050
-	-1   0    0    -1
 $EndComp
 Text Label 5600 1700 0    60   ~ 0
@@
 Wire Wire Line
 	9000 3200 8700 3200
-$Comp
-L R R13
-U 1 1 52EF83E3
-P 8900 2350
-F 0 "R13" H 8900 2450 50  0000 C CNN
-F 1 "10k" H 8900 2350 50  0000 C CNN
-F 2 "RESC1608-N" H 8900 2350 60  0001 C CNN
-F 3 "~" H 8900 2350 60  0000 C CNN
-F 4 "Yageo" H 8900 2350 60  0001 C CNN "MFR Name"
-F 5 "RC0603JR-0710KL" H 8900 2350 60  0001 C CNN "MFR Part No"
-F 6 "311-10KGRCT-ND" H 8900 2350 60  0001 C CNN "Distributor Part No"
-F 7 "0.1W" H 8900 2250 50  0001 C CNN "Power"
-F 8 "5%" H 8900 2150 50  0001 C CNN "Tolerance"
-	1    8900 2350
-	0    -1   -1   0
-$EndComp
 Wire Wire Line
 	7200 2200 7300 2200
@@
 	7000 3500 7300 3500
 $Comp
-L R R14
-U 1 1 52F2E641
-P 9250 3300
-F 0 "R14" H 9250 3400 50  0000 C CNN
-F 1 "10k" H 9250 3300 50  0000 C CNN
-F 2 "~" H 9250 3300 60  0000 C CNN
-F 3 "~" H 9250 3300 60  0000 C CNN
-F 4 "W" H 9250 3200 50  0001 C CNN "Power"
-F 5 "%" H 9250 3100 50  0001 C CNN "Tolerance"
-	1    9250 3300
-	-1   0    0    1
-$EndComp
-$Comp
 L C C24
 U 1 1 52F5954D
@@
 	1    0    0    -1
 $EndComp
+$Comp
+L C C31
+U 1 1 52F59BE8
+P 4800 2050
+F 0 "C31" H 4850 2200 60  0000 L CNN
+F 1 "22pF" H 4850 1900 60  0000 L CNN
+F 2 "CAPC1005-N" H 4800 2050 60  0001 C CNN
+F 3 "~" H 4800 2050 60  0000 C CNN
+F 4 "Yageo" H 4800 2050 60  0001 C CNN "MFR Name"
+F 5 "CC0402JRNPO9BN220" H 4800 2050 60  0001 C CNN "MFR Part No"
+F 6 "311-1018-1-ND" H 4800 2050 60  0001 C CNN "Distributor Part No"
+F 7 "50V" H 4750 1900 60  0001 R CNN "Voltage"
+F 8 "C0G" H 4750 2200 60  0001 R CNN "Dielectric"
+	1    4800 2050
+	-1   0    0    -1
+$EndComp
+$Comp
+L C C33
+U 1 1 52F59C29
+P 5500 2050
+F 0 "C33" H 5550 2200 60  0000 L CNN
+F 1 "22pF" H 5550 1900 60  0000 L CNN
+F 2 "CAPC1005-N" H 5500 2050 60  0001 C CNN
+F 3 "~" H 5500 2050 60  0000 C CNN
+F 4 "Yageo" H 5500 2050 60  0001 C CNN "MFR Name"
+F 5 "CC0402JRNPO9BN220" H 5500 2050 60  0001 C CNN "MFR Part No"
+F 6 "311-1018-1-ND" H 5500 2050 60  0001 C CNN "Distributor Part No"
+F 7 "50V" H 5450 1900 60  0001 R CNN "Voltage"
+F 8 "C0G" H 5450 2200 60  0001 R CNN "Dielectric"
+	1    5500 2050
+	1    0    0    -1
+$EndComp
+$Comp
+L R R13
+U 1 1 52F59C6E
+P 8900 2350
+F 0 "R13" H 8900 2450 50  0000 C CNN
+F 1 "10k" H 8900 2350 50  0000 C CNN
+F 2 "RESC1005-N" H 8900 2350 60  0001 C CNN
+F 3 "~" H 8900 2350 60  0000 C CNN
+F 4 "Stackpole" H 8900 2350 60  0001 C CNN "MFR Name"
+F 5 "RMCF0402JT10K0" H 8900 2350 60  0001 C CNN "MFR Part No"
+F 6 "RMCF0402JT10K0CT-ND" H 8900 2350 60  0001 C CNN "Distributor Part No"
+F 7 "1/16W" H 8900 2250 50  0001 C CNN "Power"
+F 8 "5%" H 8900 2150 50  0001 C CNN "Tolerance"
+	1    8900 2350
+	0    -1   -1   0
+$EndComp
+$Comp
+L C C34
+U 1 1 52F59E18
+P 7550 2200
+F 0 "C34" H 7600 2350 60  0000 L CNN
+F 1 "0.1uF" H 7600 2050 60  0000 L CNN
+F 2 "CAPC1005-N" H 7550 2200 60  0001 C CNN
+F 3 "~" H 7550 2200 60  0000 C CNN
+F 4 "Samsung" H 7550 2200 60  0001 C CNN "MFR Name"
+F 5 "CL05B104KO5NNNC" H 7550 2200 60  0001 C CNN "MFR Part No"
+F 6 "1276-1001-1-ND" H 7550 2200 60  0001 C CNN "Distributor Part No"
+F 7 "16V" H 7500 2050 60  0001 R CNN "Voltage"
+F 8 "X7R" H 7500 2350 60  0001 R CNN "Dielectric"
+	1    7550 2200
+	0    -1   -1   0
+$EndComp
+$Comp
+L R R14
+U 1 1 52F59E59
+P 9250 3300
+F 0 "R14" H 9250 3400 50  0000 C CNN
+F 1 "10k" H 9250 3300 50  0000 C CNN
+F 2 "RESC1005-N" H 9250 3300 60  0001 C CNN
+F 3 "~" H 9250 3300 60  0000 C CNN
+F 4 "Stackpole" H 9250 3300 60  0001 C CNN "MFR Name"
+F 5 "RMCF0402JT10K0" H 9250 3300 60  0001 C CNN "MFR Part No"
+F 6 "RMCF0402JT10K0CT-ND" H 9250 3300 60  0001 C CNN "Distributor Part No"
+F 7 "1/16W" H 9250 3200 50  0001 C CNN "Power"
+F 8 "5%" H 9250 3100 50  0001 C CNN "Tolerance"
+	1    9250 3300
+	-1   0    0    1
+$EndComp
+Wire Wire Line
+	9500 3300 9600 3300
 $EndSCHEMATC
