File: Hardware/GPS.sch (KiCad schematic (older format))
At the start: 15 parts

Commit message: GPS values
Parts:
- removed C? (x4): 22pF, ~, symbol C
- removed C?: C, ~, symbol C
- removed L?: L, ~, symbol L
- removed R?: R, ~, symbol R
- added C4: 4.7uF, CAPC2012-N, symbol C
- added C6, C7, C8, C9: 22pF, CAPC1005-N, symbol C
- added L3: DNP, INDC1005-N, symbol L
- added R2: 10k, RESC1608-N, symbol R
- C10: renamed from C?; footprint ~ -> CAPC1005-N; Dielectric D -> NP0; Distributor Part No (none) -> 311-1415-1-ND; MFR Name (none) -> Yageo; MFR Part No (none) -> CC0402JRNPO9BN180; Voltage V -> 50V
- C5: renamed from C?; footprint ~ -> CAPC1005-N; Dielectric D -> C0G; Distributor Part No (none) -> 311-1018-1-ND; MFR Name (none) -> Yageo; MFR Part No (none) -> CC0402JRNPO9BN220; Voltage V -> 50V
- L2: renamed from L?; value L -> DNP; footprint ~ -> INDC1005-N
- Q1: renamed from Q?; value MOSFET-P -> IRLML6401; footprint ~ -> SOT95P280-3N-GDS; Distributor Part No (none) -> IRLML6401PBFCT-ND; MFR Name (none) -> IR; MFR Part No (none) -> IRLML6401TRPBF
- R3: renamed from R?; value R -> 100; footprint ~ -> RESC1608-N; Distributor Part No (none) -> 311-100GRCT-ND; MFR Name (none) -> Yageo; MFR Part No (none) -> RC0603JR-07100RL; Power W -> 0.1W; Tolerance % -> 5%
- gave numbers to parts that had none: 3
Connections:
- net +3.3V: now also C7.1, R2.2
- net GND: now also C4.2, C6.2, C7.2, C8.2, C9.2, L3.2
- net GPS_En: now also R2.1
- net at FB1.2, U2.11 (TX): now also C8.1
- net at FB2.2, U2.13 (RX): now also C9.1
- net at C5.1, Q1.D, U2.25 (VddRF)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: now also C4.1, C6.1
- net at C10.2, U2.3 (AntOut): now also L3.1
Changed lines of the file:
@@
 $EndDescr
 $Comp
-L ANTENOVA-UB U?
+L ANTENOVA-UB U2
 U 1 1 52E9B1BE
 P 7100 4150
-F 0 "U?" H 7100 5300 60  0000 C CNN
+F 0 "U2" H 7100 5300 60  0000 C CNN
 F 1 "ANTENOVA-UB" H 7100 3000 60  0000 C CNN
 F 2 "~" H 7100 4150 60  0000 C CNN
@@
 $EndComp
 $Comp
-L C C?
+L C C10
 U 1 1 52E9B2C1
 P 7900 3450
-F 0 "C?" H 7950 3600 60  0000 L CNN
+F 0 "C10" H 7950 3600 60  0000 L CNN
 F 1 "18pF" H 7950 3300 60  0000 L CNN
-F 2 "~" H 7900 3450 60  0000 C CNN
+F 2 "CAPC1005-N" H 7900 3450 60  0001 C CNN
 F 3 "~" H 7900 3450 60  0000 C CNN
-F 4 "V" H 7850 3300 60  0001 R CNN "Voltage"
-F 5 "D" H 7850 3600 60  0001 R CNN "Dielectric"
+F 4 "Yageo" H 7900 3450 60  0001 C CNN "MFR Name"
+F 5 "CC0402JRNPO9BN180" H 7900 3450 60  0001 C CNN "MFR Part No"
+F 6 "311-1415-1-ND" H 7900 3450 60  0001 C CNN "Distributor Part No"
+F 7 "50V" H 7850 3300 60  0001 R CNN "Voltage"
+F 8 "NP0" H 7850 3600 60  0001 R CNN "Dielectric"
 	1    7900 3450
 	1    0    0    -1
 $EndComp
 $Comp
-L L L?
+L L L2
 U 1 1 52E9B2DC
 P 8350 3100
-F 0 "L?" H 8350 3000 60  0000 C CNN
-F 1 "L" H 8350 3150 60  0000 C CNN
-F 2 "~" H 8350 3100 60  0000 C CNN
+F 0 "L2" H 8350 3000 60  0000 C CNN
+F 1 "DNP" H 8350 3150 60  0000 C CNN
+F 2 "INDC1005-N" H 8350 3100 60  0001 C CNN
 F 3 "~" H 8350 3100 60  0000 C CNN
 	1    8350 3100
-	1    0    0    -1
-$EndComp
-$Comp
-L L L?
-U 1 1 52E9B2EB
-P 8350 3800
-F 0 "L?" H 8350 3700 60  0000 C CNN
-F 1 "L" H 8350 3850 60  0000 C CNN
-F 2 "~" H 8350 3800 60  0000 C CNN
-F 3 "~" H 8350 3800 60  0000 C CNN
-	1    8350 3800
 	1    0    0    -1
 $EndComp
@@
 $EndComp
 $Comp
-L FERRITE FB?
+L FERRITE FB1
 U 1 1 52E9B435
 P 5150 4200
-F 0 "FB?" H 5100 4250 60  0000 R CNN
+F 0 "FB1" H 5100 4250 60  0000 R CNN
 F 1 "1k" H 5200 4150 60  0000 L CNN
 F 2 "RESC1005-N" H 5150 4200 60  0001 C CNN
@@
 $EndComp
 $Comp
-L FERRITE FB?
+L FERRITE FB2
 U 1 1 52E9B565
 P 5150 4500
-F 0 "FB?" H 5100 4550 60  0000 R CNN
+F 0 "FB2" H 5100 4550 60  0000 R CNN
 F 1 "1k" H 5200 4450 60  0000 L CNN
 F 2 "RESC1005-N" H 5150 4500 60  0001 C CNN
@@
 	1    0    0    -1
 $EndComp
-$Comp
-L C C?
-U 1 1 52E9B5D4
-P 5700 3650
-F 0 "C?" H 5750 3800 60  0000 L CNN
-F 1 "22pF" H 5750 3500 60  0000 L CNN
-F 2 "~" H 5700 3650 60  0000 C CNN
-F 3 "~" H 5700 3650 60  0000 C CNN
-F 4 "V" H 5650 3500 60  0001 R CNN "Voltage"
-F 5 "D" H 5650 3800 60  0001 R CNN "Dielectric"
-	1    5700 3650
-	-1   0    0    -1
-$EndComp
 Wire Wire Line
 	8700 3800 8600 3800
@@
 Connection ~ 6400 3300
 $Comp
-L C C?
+L C C5
 U 1 1 52E9B693
 P 5300 3550
-F 0 "C?" H 5350 3700 60  0000 L CNN
+F 0 "C5" H 5350 3700 60  0000 L CNN
 F 1 "22pF" H 5350 3400 60  0000 L CNN
-F 2 "~" H 5300 3550 60  0000 C CNN
+F 2 "CAPC1005-N" H 5300 3550 60  0001 C CNN
 F 3 "~" H 5300 3550 60  0000 C CNN
-F 4 "V" H 5250 3400 60  0001 R CNN "Voltage"
-F 5 "D" H 5250 3700 60  0001 R CNN "Dielectric"
+F 4 "Yageo" H 5300 3550 60  0001 C CNN "MFR Name"
+F 5 "CC0402JRNPO9BN220" H 5300 3550 60  0001 C CNN "MFR Part No"
+F 6 "311-1018-1-ND" H 5300 3550 60  0001 C CNN "Distributor Part No"
+F 7 "50V" H 5250 3400 60  0001 R CNN "Voltage"
+F 8 "C0G" H 5250 3700 60  0001 R CNN "Dielectric"
 	1    5300 3550
 	-1   0    0    -1
@@
 NoConn ~ 6500 5000
 NoConn ~ 6500 5100
-$Comp
-L C C?
-U 1 1 52E9B6E2
-P 6100 4850
-F 0 "C?" H 6150 5000 60  0000 L CNN
-F 1 "22pF" H 6150 4700 60  0000 L CNN
-F 2 "~" H 6100 4850 60  0000 C CNN
-F 3 "~" H 6100 4850 60  0000 C CNN
-F 4 "V" H 6050 4700 60  0001 R CNN "Voltage"
-F 5 "D" H 6050 5000 60  0001 R CNN "Dielectric"
-	1    6100 4850
-	-1   0    0    -1
-$EndComp
-$Comp
-L C C?
-U 1 1 52E9B6EA
-P 5700 4850
-F 0 "C?" H 5750 5000 60  0000 L CNN
-F 1 "22pF" H 5750 4700 60  0000 L CNN
-F 2 "~" H 5700 4850 60  0000 C CNN
-F 3 "~" H 5700 4850 60  0000 C CNN
-F 4 "V" H 5650 4700 60  0001 R CNN "Voltage"
-F 5 "D" H 5650 5000 60  0001 R CNN "Dielectric"
-	1    5700 4850
-	-1   0    0    -1
-$EndComp
 Wire Wire Line
 	5700 4600 5700 4300
@@
 Text HLabel 3400 3500 0    60   Input ~ 0
 GPS_En
-$Comp
-L C C?
-U 1 1 52ECD78D
-P 6100 3850
-F 0 "C?" H 6150 4000 60  0000 L CNN
-F 1 "22pF" H 6150 3700 60  0000 L CNN
-F 2 "~" H 6100 3850 60  0000 C CNN
-F 3 "~" H 6100 3850 60  0000 C CNN
-F 4 "V" H 6050 3700 60  0001 R CNN "Voltage"
-F 5 "D" H 6050 4000 60  0001 R CNN "Dielectric"
-	1    6100 3850
-	-1   0    0    -1
-$EndComp
 $Comp
 L GND #PWR?
@@
 	5300 3100 5300 3300
 $Comp
-L MOSFET-P Q?
+L MOSFET-P Q1
 U 1 1 52EF2A40
 P 4300 3200
-F 0 "Q?" H 4200 3150 60  0000 R CNN
-F 1 "MOSFET-P" V 4500 3200 60  0000 C CNN
-F 2 "~" H 4300 3200 60  0000 C CNN
+F 0 "Q1" H 4200 3150 60  0000 R CNN
+F 1 "IRLML6401" V 4500 3200 60  0000 C CNN
+F 2 "SOT95P280-3N-GDS" H 4300 3200 60  0001 C CNN
 F 3 "~" H 4300 3200 60  0000 C CNN
+F 4 "IR" H 4300 3200 60  0001 C CNN "MFR Name"
+F 5 "IRLML6401TRPBF" H 4300 3200 60  0001 C CNN "MFR Part No"
+F 6 "IRLML6401PBFCT-ND" H 4300 3200 60  0001 C CNN "Distributor Part No"
 	1    4300 3200
 	0    -1   -1   0
 $EndComp
 $Comp
-L R R?
+L R R3
 U 1 1 52EF2A4F
 P 3850 3500
-F 0 "R?" H 3850 3600 50  0000 C CNN
-F 1 "R" H 3850 3500 50  0000 C CNN
-F 2 "~" H 3850 3500 60  0000 C CNN
+F 0 "R3" H 3850 3600 50  0000 C CNN
+F 1 "100" H 3850 3500 50  0000 C CNN
+F 2 "RESC1608-N" H 3850 3500 60  0001 C CNN
 F 3 "~" H 3850 3500 60  0000 C CNN
-F 4 "W" H 3850 3400 50  0001 C CNN "Power"
-F 5 "%" H 3850 3300 50  0001 C CNN "Tolerance"
+F 4 "Yageo" H 3850 3500 60  0001 C CNN "MFR Name"
+F 5 "RC0603JR-07100RL" H 3850 3500 60  0001 C CNN "MFR Part No"
+F 6 "311-100GRCT-ND" H 3850 3500 60  0001 C CNN "Distributor Part No"
+F 7 "0.1W" H 3850 3400 50  0001 C CNN "Power"
+F 8 "5%" H 3850 3300 50  0001 C CNN "Tolerance"
 	1    3850 3500
 	1    0    0    -1
-$EndComp
-$Comp
-L C C?
-U 1 1 52EF2A6A
-P 4900 3450
-F 0 "C?" H 4950 3600 60  0000 L CNN
-F 1 "C" H 4950 3300 60  0000 L CNN
-F 2 "~" H 4900 3450 60  0000 C CNN
-F 3 "~" H 4900 3450 60  0000 C CNN
-F 4 "V" H 4850 3300 60  0001 R CNN "Voltage"
-F 5 "D" H 4850 3600 60  0001 R CNN "Dielectric"
-	1    4900 3450
-	-1   0    0    -1
 $EndComp
 $Comp
@@
 Wire Wire Line
 	4200 3500 4100 3500
-$Comp
-L R R?
-U 1 1 52EF2C24
-P 3500 3150
-F 0 "R?" H 3500 3250 50  0000 C CNN
-F 1 "R" H 3500 3150 50  0000 C CNN
-F 2 "~" H 3500 3150 60  0000 C CNN
-F 3 "~" H 3500 3150 60  0000 C CNN
-F 4 "W" H 3500 3050 50  0001 C CNN "Power"
-F 5 "%" H 3500 2950 50  0001 C CNN "Tolerance"
-	1    3500 3150
-	0    -1   -1   0
-$EndComp
 Wire Wire Line
 	3400 3500 3600 3500
@@
 	3800 3100 4100 3100
 Connection ~ 3500 2800
+$Comp
+L C C4
+U 1 1 52EF664A
+P 4900 3450
+F 0 "C4" H 4950 3600 60  0000 L CNN
+F 1 "4.7uF" H 4950 3300 60  0000 L CNN
+F 2 "CAPC2012-N" H 4900 3450 60  0001 C CNN
+F 3 "~" H 4900 3450 60  0000 C CNN
+F 4 "Samsung" H 4900 3450 60  0001 C CNN "MFR Name"
+F 5 "CL21A475KOFNNNE" H 4900 3450 60  0001 C CNN "MFR Part No"
+F 6 "1276-1065-1-ND" H 4900 3450 60  0001 C CNN "Distributor Part No"
+F 7 "16V" H 4850 3300 60  0001 R CNN "Voltage"
+F 8 "X5R" H 4850 3600 60  0001 R CNN "Dielectric"
+	1    4900 3450
+	-1   0    0    -1
+$EndComp
+$Comp
+L R R2
+U 1 1 52EF67CC
+P 3500 3150
+F 0 "R2" H 3500 3250 50  0000 C CNN
+F 1 "10k" H 3500 3150 50  0000 C CNN
+F 2 "RESC1608-N" H 3500 3150 60  0001 C CNN
+F 3 "~" H 3500 3150 60  0000 C CNN
+F 4 "Yageo" H 3500 3150 60  0001 C CNN "MFR Name"
+F 5 "RC0603JR-0710KL" H 3500 3150 60  0001 C CNN "MFR Part No"
+F 6 "311-10KGRCT-ND" H 3500 3150 60  0001 C CNN "Distributor Part No"
+F 7 "0.1W" H 3500 3050 50  0001 C CNN "Power"
+F 8 "5%" H 3500 2950 50  0001 C CNN "Tolerance"
+	1    3500 3150
+	0    -1   -1   0
+$EndComp
+$Comp
+L C C6
+U 1 1 52EF6821
+P 5700 3650
+F 0 "C6" H 5750 3800 60  0000 L CNN
+F 1 "22pF" H 5750 3500 60  0000 L CNN
+F 2 "CAPC1005-N" H 5700 3650 60  0001 C CNN
+F 3 "~" H 5700 3650 60  0000 C CNN
+F 4 "Yageo" H 5700 3650 60  0001 C CNN "MFR Name"
+F 5 "CC0402JRNPO9BN220" H 5700 3650 60  0001 C CNN "MFR Part No"
+F 6 "311-1018-1-ND" H 5700 3650 60  0001 C CNN "Distributor Part No"
+F 7 "50V" H 5650 3500 60  0001 R CNN "Voltage"
+F 8 "C0G" H 5650 3800 60  0001 R CNN "Dielectric"
+	1    5700 3650
+	-1   0    0    -1
+$EndComp
+$Comp
+L C C7
+U 1 1 52EF682C
+P 6100 3850
+F 0 "C7" H 6150 4000 60  0000 L CNN
+F 1 "22pF" H 6150 3700 60  0000 L CNN
+F 2 "CAPC1005-N" H 6100 3850 60  0001 C CNN
+F 3 "~" H 6100 3850 60  0000 C CNN
+F 4 "Yageo" H 6100 3850 60  0001 C CNN "MFR Name"
+F 5 "CC0402JRNPO9BN220" H 6100 3850 60  0001 C CNN "MFR Part No"
+F 6 "311-1018-1-ND" H 6100 3850 60  0001 C CNN "Distributor Part No"
+F 7 "50V" H 6050 3700 60  0001 R CNN "Voltage"
+F 8 "C0G" H 6050 4000 60  0001 R CNN "Dielectric"
+	1    6100 3850
+	-1   0    0    -1
+$EndComp
+$Comp
+L C C8
+U 1 1 52EF6837
+P 5700 4850
+F 0 "C8" H 5750 5000 60  0000 L CNN
+F 1 "22pF" H 5750 4700 60  0000 L CNN
+F 2 "CAPC1005-N" H 5700 4850 60  0001 C CNN
+F 3 "~" H 5700 4850 60  0000 C CNN
+F 4 "Yageo" H 5700 4850 60  0001 C CNN "MFR Name"
+F 5 "CC0402JRNPO9BN220" H 5700 4850 60  0001 C CNN "MFR Part No"
+F 6 "311-1018-1-ND" H 5700 4850 60  0001 C CNN "Distributor Part No"
+F 7 "50V" H 5650 4700 60  0001 R CNN "Voltage"
+F 8 "C0G" H 5650 5000 60  0001 R CNN "Dielectric"
+	1    5700 4850
+	-1   0    0    -1
+$EndComp
+$Comp
+L C C9
+U 1 1 52EF6842
+P 6100 4850
+F 0 "C9" H 6150 5000 60  0000 L CNN
+F 1 "22pF" H 6150 4700 60  0000 L CNN
+F 2 "CAPC1005-N" H 6100 4850 60  0001 C CNN
+F 3 "~" H 6100 4850 60  0000 C CNN
+F 4 "Yageo" H 6100 4850 60  0001 C CNN "MFR Name"
+F 5 "CC0402JRNPO9BN220" H 6100 4850 60  0001 C CNN "MFR Part No"
+F 6 "311-1018-1-ND" H 6100 4850 60  0001 C CNN "Distributor Part No"
+F 7 "50V" H 6050 4700 60  0001 R CNN "Voltage"
+F 8 "C0G" H 6050 5000 60  0001 R CNN "Dielectric"
+	1    6100 4850
+	-1   0    0    -1
+$EndComp
+$Comp
+L L L3
+U 1 1 52EF6969
+P 8350 3800
+F 0 "L3" H 8350 3700 60  0000 C CNN
+F 1 "DNP" H 8350 3850 60  0000 C CNN
+F 2 "INDC1005-N" H 8350 3800 60  0001 C CNN
+F 3 "~" H 8350 3800 60  0000 C CNN
+	1    8350 3800
+	1    0    0    -1
+$EndComp
 $EndSCHEMATC

Commit message: Something changed
Parts:
- renumbered C4 to C1, C5 to C2, C6 to C3, C8 to C4, C7 to C5, C9 to C6, C10 to C7, L2 to L1, L3 to L2, R2 to R3, R3 to R4, U2 to U1
Changed lines of the file:
@@
 Sheet 2 4
 Title "Aether - Pico Tracker"
-Date "3 feb 2014"
+Date "4 feb 2014"
 Rev "1"
 Comp "Aerodyne Labs"
@@
 $EndDescr
 $Comp
-L ANTENOVA-UB U2
+L ANTENOVA-UB U1
 U 1 1 52E9B1BE
 P 7100 4150
-F 0 "U2" H 7100 5300 60  0000 C CNN
+F 0 "U1" H 7100 5300 60  0000 C CNN
 F 1 "ANTENOVA-UB" H 7100 3000 60  0000 C CNN
 F 2 "~" H 7100 4150 60  0000 C CNN
@@
 $EndComp
 $Comp
-L C C10
+L C C7
 U 1 1 52E9B2C1
 P 7900 3450
-F 0 "C10" H 7950 3600 60  0000 L CNN
+F 0 "C7" H 7950 3600 60  0000 L CNN
 F 1 "18pF" H 7950 3300 60  0000 L CNN
 F 2 "CAPC1005-N" H 7900 3450 60  0001 C CNN
@@
 $EndComp
 $Comp
-L L L2
+L L L1
 U 1 1 52E9B2DC
 P 8350 3100
-F 0 "L2" H 8350 3000 60  0000 C CNN
+F 0 "L1" H 8350 3000 60  0000 C CNN
 F 1 "DNP" H 8350 3150 60  0000 C CNN
 F 2 "INDC1005-N" H 8350 3100 60  0001 C CNN
@@
 $EndComp
 $Comp
-L GND #PWR?
+L GND #PWR08
 U 1 1 52E9B2FA
 P 8700 3100
-F 0 "#PWR?" H 8700 3100 30  0001 C CNN
+F 0 "#PWR08" H 8700 3100 30  0001 C CNN
 F 1 "GND" H 8700 3030 30  0001 C CNN
 F 2 "" H 8700 3100 60  0000 C CNN
@@
 $EndComp
 $Comp
-L GND #PWR?
+L GND #PWR09
 U 1 1 52E9B317
 P 8700 3800
-F 0 "#PWR?" H 8700 3800 30  0001 C CNN
+F 0 "#PWR09" H 8700 3800 30  0001 C CNN
 F 1 "GND" H 8700 3730 30  0001 C CNN
 F 2 "" H 8700 3800 60  0000 C CNN
@@
 $EndComp
 $Comp
-L GND #PWR?
+L GND #PWR010
 U 1 1 52E9B346
 P 7800 5300
-F 0 "#PWR?" H 7800 5300 30  0001 C CNN
+F 0 "#PWR010" H 7800 5300 30  0001 C CNN
 F 1 "GND" H 7800 5230 30  0001 C CNN
 F 2 "" H 7800 5300 60  0000 C CNN
@@
 NoConn ~ 6500 3800
 $Comp
-L GND #PWR?
+L GND #PWR011
 U 1 1 52E9B409
 P 6400 5300
-F 0 "#PWR?" H 6400 5300 30  0001 C CNN
+F 0 "#PWR011" H 6400 5300 30  0001 C CNN
 F 1 "GND" H 6400 5230 30  0001 C CNN
 F 2 "" H 6400 5300 60  0000 C CNN
@@
 Connection ~ 6400 3300
 $Comp
-L C C5
+L C C2
 U 1 1 52E9B693
 P 5300 3550
-F 0 "C5" H 5350 3700 60  0000 L CNN
+F 0 "C2" H 5350 3700 60  0000 L CNN
 F 1 "22pF" H 5350 3400 60  0000 L CNN
 F 2 "CAPC1005-N" H 5300 3550 60  0001 C CNN
@@
 Connection ~ 6100 4400
 $Comp
-L GND #PWR?
+L GND #PWR012
 U 1 1 52E9B758
 P 5700 5200
-F 0 "#PWR?" H 5700 5200 30  0001 C CNN
+F 0 "#PWR012" H 5700 5200 30  0001 C CNN
 F 1 "GND" H 5700 5130 30  0001 C CNN
 F 2 "" H 5700 5200 60  0000 C CNN
@@
 $EndComp
 $Comp
-L GND #PWR?
+L GND #PWR013
 U 1 1 52E9B767
 P 6100 5200
-F 0 "#PWR?" H 6100 5200 30  0001 C CNN
+F 0 "#PWR013" H 6100 5200 30  0001 C CNN
 F 1 "GND" H 6100 5130 30  0001 C CNN
 F 2 "" H 6100 5200 60  0000 C CNN
@@
 	4900 4500 4700 4500
 $Comp
-L GND #PWR?
+L GND #PWR014
 U 1 1 52E9B83C
 P 5700 4000
-F 0 "#PWR?" H 5700 4000 30  0001 C CNN
+F 0 "#PWR014" H 5700 4000 30  0001 C CNN
 F 1 "GND" H 5700 3930 30  0001 C CNN
 F 2 "" H 5700 4000 60  0000 C CNN
@@
 $EndComp
 $Comp
-L GND #PWR?
+L GND #PWR015
 U 1 1 52E9B84B
 P 5300 3900
-F 0 "#PWR?" H 5300 3900 30  0001 C CNN
+F 0 "#PWR015" H 5300 3900 30  0001 C CNN
 F 1 "GND" H 5300 3830 30  0001 C CNN
 F 2 "" H 5300 3900 60  0000 C CNN
@@
 GPS_En
 $Comp
-L GND #PWR?
+L GND #PWR016
 U 1 1 52ECD7A8
 P 6100 4200
-F 0 "#PWR?" H 6100 4200 30  0001 C CNN
+F 0 "#PWR016" H 6100 4200 30  0001 C CNN
 F 1 "GND" H 6100 4130 30  0001 C CNN
 F 2 "" H 6100 4200 60  0000 C CNN
@@
 	6100 3000 6100 3600
 $Comp
-L +3.3V #PWR?
+L +3.3V #PWR017
 U 1 1 52ECD869
 P 6100 3000
-F 0 "#PWR?" H 6100 2960 30  0001 C CNN
+F 0 "#PWR017" H 6100 2960 30  0001 C CNN
 F 1 "+3.3V" H 6100 3110 30  0000 C CNN
 F 2 "" H 6100 3000 60  0000 C CNN
@@
 $EndComp
 $Comp
-L R R3
+L R R4
 U 1 1 52EF2A4F
 P 3850 3500
-F 0 "R3" H 3850 3600 50  0000 C CNN
+F 0 "R4" H 3850 3600 50  0000 C CNN
 F 1 "100" H 3850 3500 50  0000 C CNN
 F 2 "RESC1608-N" H 3850 3500 60  0001 C CNN
@@
 $EndComp
 $Comp
-L GND #PWR?
+L GND #PWR018
 U 1 1 52EF2A9A
 P 4900 3800
-F 0 "#PWR?" H 4900 3800 30  0001 C CNN
+F 0 "#PWR018" H 4900 3800 30  0001 C CNN
 F 1 "GND" H 4900 3730 30  0001 C CNN
 F 2 "" H 4900 3800 60  0000 C CNN
@@
 Connection ~ 3500 3500
 $Comp
-L +3.3V #PWR?
+L +3.3V #PWR019
 U 1 1 52EF2CCE
 P 3500 2700
-F 0 "#PWR?" H 3500 2660 30  0001 C CNN
+F 0 "#PWR019" H 3500 2660 30  0001 C CNN
 F 1 "+3.3V" H 3500 2810 30  0000 C CNN
 F 2 "" H 3500 2700 60  0000 C CNN
@@
 Connection ~ 3500 2800
 $Comp
-L C C4
+L C C1
 U 1 1 52EF664A
 P 4900 3450
-F 0 "C4" H 4950 3600 60  0000 L CNN
+F 0 "C1" H 4950 3600 60  0000 L CNN
 F 1 "4.7uF" H 4950 3300 60  0000 L CNN
 F 2 "CAPC2012-N" H 4900 3450 60  0001 C CNN
@@
 $EndComp
 $Comp
-L R R2
+L R R3
 U 1 1 52EF67CC
 P 3500 3150
-F 0 "R2" H 3500 3250 50  0000 C CNN
+F 0 "R3" H 3500 3250 50  0000 C CNN
 F 1 "10k" H 3500 3150 50  0000 C CNN
 F 2 "RESC1608-N" H 3500 3150 60  0001 C CNN
@@
 $EndComp
 $Comp
-L C C6
+L C C3
 U 1 1 52EF6821
 P 5700 3650
-F 0 "C6" H 5750 3800 60  0000 L CNN
+F 0 "C3" H 5750 3800 60  0000 L CNN
 F 1 "22pF" H 5750 3500 60  0000 L CNN
 F 2 "CAPC1005-N" H 5700 3650 60  0001 C CNN
@@
 $EndComp
 $Comp
-L C C7
+L C C5
 U 1 1 52EF682C
 P 6100 3850
-F 0 "C7" H 6150 4000 60  0000 L CNN
+F 0 "C5" H 6150 4000 60  0000 L CNN
 F 1 "22pF" H 6150 3700 60  0000 L CNN
 F 2 "CAPC1005-N" H 6100 3850 60  0001 C CNN
@@
 $EndComp
 $Comp
-L C C8
+L C C4
 U 1 1 52EF6837
 P 5700 4850
-F 0 "C8" H 5750 5000 60  0000 L CNN
+F 0 "C4" H 5750 5000 60  0000 L CNN
 F 1 "22pF" H 5750 4700 60  0000 L CNN
 F 2 "CAPC1005-N" H 5700 4850 60  0001 C CNN
@@
 $EndComp
 $Comp
-L C C9
+L C C6
 U 1 1 52EF6842
 P 6100 4850
-F 0 "C9" H 6150 5000 60  0000 L CNN
+F 0 "C6" H 6150 5000 60  0000 L CNN
 F 1 "22pF" H 6150 4700 60  0000 L CNN
 F 2 "CAPC1005-N" H 6100 4850 60  0001 C CNN
@@
 $EndComp
 $Comp
-L L L3
+L L L2
 U 1 1 52EF6969
 P 8350 3800
-F 0 "L3" H 8350 3700 60  0000 C CNN
+F 0 "L2" H 8350 3700 60  0000 C CNN
 F 1 "DNP" H 8350 3850 60  0000 C CNN
 F 2 "INDC1005-N" H 8350 3800 60  0001 C CNN
