File: Hardware/GPS.sch (KiCad schematic (older format))
At the start: 15 parts, among them Q1 IRLML6401, U1 ANTENOVA-UB

Commit message: GPS components
Parts:
- R3: footprint RESC1608-N -> RESC1005-N; Distributor Part No 311-10KGRCT-ND -> RMCF0402JT10K0CT-ND; MFR Name Yageo -> Stackpole; MFR Part No RC0603JR-0710KL -> RMCF0402JT10K0; Power 0.1W -> 1/16W
- R4: footprint RESC1608-N -> RESC1005-N; Distributor Part No 311-100GRCT-ND -> 311-100JRCT-ND; MFR Part No RC0603JR-07100RL -> RC0402JR-07100RL; Power 0.1W -> 1/16W
Changed lines of the file:
@@
 F 0 "R4" H 3850 3600 50  0000 C CNN
 F 1 "100" H 3850 3500 50  0000 C CNN
-F 2 "RESC1608-N" H 3850 3500 60  0001 C CNN
+F 2 "RESC1005-N" H 3850 3500 60  0001 C CNN
 F 3 "~" H 3850 3500 60  0000 C CNN
 F 4 "Yageo" H 3850 3500 60  0001 C CNN "MFR Name"
-F 5 "RC0603JR-07100RL" H 3850 3500 60  0001 C CNN "MFR Part No"
-F 6 "311-100GRCT-ND" H 3850 3500 60  0001 C CNN "Distributor Part No"
-F 7 "0.1W" H 3850 3400 50  0001 C CNN "Power"
+F 5 "RC0402JR-07100RL" H 3850 3500 60  0001 C CNN "MFR Part No"
+F 6 "311-100JRCT-ND" H 3850 3500 60  0001 C CNN "Distributor Part No"
+F 7 "1/16W" H 3850 3400 50  0001 C CNN "Power"
 F 8 "5%" H 3850 3300 50  0001 C CNN "Tolerance"
 	1    3850 3500
@@
 	1    4900 3450
 	-1   0    0    -1
-$EndComp
-$Comp
-L R R3
-U 1 1 52EF67CC
-P 3500 3150
-F 0 "R3" H 3500 3250 50  0000 C CNN
-F 1 "10k" H 3500 3150 50  0000 C CNN
-F 2 "RESC1608-N" H 3500 3150 60  0001 C CNN
-F 3 "~" H 3500 3150 60  0000 C CNN
-F 4 "Yageo" H 3500 3150 60  0001 C CNN "MFR Name"
-F 5 "RC0603JR-0710KL" H 3500 3150 60  0001 C CNN "MFR Part No"
-F 6 "311-10KGRCT-ND" H 3500 3150 60  0001 C CNN "Distributor Part No"
-F 7 "0.1W" H 3500 3050 50  0001 C CNN "Power"
-F 8 "5%" H 3500 2950 50  0001 C CNN "Tolerance"
-	1    3500 3150
-	0    -1   -1   0
 $EndComp
 $Comp
@@
 	1    0    0    -1
 $EndComp
+$Comp
+L R R3
+U 1 1 52F5BCF8
+P 3500 3150
+F 0 "R3" H 3500 3250 50  0000 C CNN
+F 1 "10k" H 3500 3150 50  0000 C CNN
+F 2 "RESC1005-N" H 3500 3150 60  0001 C CNN
+F 3 "~" H 3500 3150 60  0000 C CNN
+F 4 "Stackpole" H 3500 3150 60  0001 C CNN "MFR Name"
+F 5 "RMCF0402JT10K0" H 3500 3150 60  0001 C CNN "MFR Part No"
+F 6 "RMCF0402JT10K0CT-ND" H 3500 3150 60  0001 C CNN "Distributor Part No"
+F 7 "1/16W" H 3500 3050 50  0001 C CNN "Power"
+F 8 "5%" H 3500 2950 50  0001 C CNN "Tolerance"
+	1    3500 3150
+	0    -1   -1   0
+$EndComp
 $EndSCHEMATC

Commit message: Consolidate LED resistors
See #1
Parts:
- R4: value 100 -> 120; footprint RESC1005-N -> RESC1005_N; Distributor Part No 311-100JRCT-ND -> 1276-4354-1-ND; MFR Name Yageo -> Samsung; MFR Part No RC0402JR-07100RL -> RC1005J121CS
Changed lines of the file:
@@
 $Descr A4 11693 8268
 encoding utf-8
-Sheet 2 4
+Sheet 4 4
 Title "Aether - Pico Tracker"
-Date "9 feb 2014"
+Date "24 feb 2014"
 Rev "1"
 Comp "Aerodyne Labs"
@@
 $EndComp
 $Comp
-L R R4
-U 1 1 52EF2A4F
-P 3850 3500
-F 0 "R4" H 3850 3600 50  0000 C CNN
-F 1 "100" H 3850 3500 50  0000 C CNN
-F 2 "RESC1005-N" H 3850 3500 60  0001 C CNN
-F 3 "~" H 3850 3500 60  0000 C CNN
-F 4 "Yageo" H 3850 3500 60  0001 C CNN "MFR Name"
-F 5 "RC0402JR-07100RL" H 3850 3500 60  0001 C CNN "MFR Part No"
-F 6 "311-100JRCT-ND" H 3850 3500 60  0001 C CNN "Distributor Part No"
-F 7 "1/16W" H 3850 3400 50  0001 C CNN "Power"
-F 8 "5%" H 3850 3300 50  0001 C CNN "Tolerance"
-	1    3850 3500
-	1    0    0    -1
-$EndComp
-$Comp
 L GND #PWR065
 U 1 1 52EF2A9A
@@
 	0    -1   -1   0
 $EndComp
+$Comp
+L R R4
+U 1 1 530ACEAC
+P 3850 3500
+F 0 "R4" H 3850 3600 50  0000 C CNN
+F 1 "120" H 3850 3500 50  0000 C CNN
+F 2 "RESC1005_N" H 3850 3500 60  0001 C CNN
+F 3 "~" H 3850 3500 60  0000 C CNN
+F 4 "Samsung" H 3850 3500 60  0001 C CNN "MFR Name"
+F 5 "RC1005J121CS" H 3850 3500 60  0001 C CNN "MFR Part No"
+F 6 "1276-4354-1-ND" H 3850 3500 60  0001 C CNN "Distributor Part No"
+F 7 "1/16W" H 3850 3400 50  0001 C CNN "Power"
+F 8 "5%" H 3850 3300 50  0001 C CNN "Tolerance"
+	1    3850 3500
+	1    0    0    -1
+$EndComp
 $EndSCHEMATC

Commit message: Consolidate audio filter
Consolidate pull up resistors and audio filter.
Consolidate loop filter capacitor and audio filter.
See #1
Parts:
- R3: Distributor Part No RMCF0402JT10K0CT-ND -> 311-10.0KLRCT-ND; MFR Name Stackpole -> Yageo; MFR Part No RMCF0402JT10K0 -> RC0402FR-0710KL; Tolerance 5% -> 1%
Changed lines of the file:
@@
-$EndComp
-$Comp
-L R R3
-U 1 1 52F5BCF8
-P 3500 3150
-F 0 "R3" H 3500 3250 50  0000 C CNN
-F 1 "10k" H 3500 3150 50  0000 C CNN
-F 2 "RESC1005-N" H 3500 3150 60  0001 C CNN
-F 3 "~" H 3500 3150 60  0000 C CNN
-F 4 "Stackpole" H 3500 3150 60  0001 C CNN "MFR Name"
-F 5 "RMCF0402JT10K0" H 3500 3150 60  0001 C CNN "MFR Part No"
-F 6 "RMCF0402JT10K0CT-ND" H 3500 3150 60  0001 C CNN "Distributor Part No"
-F 7 "1/16W" H 3500 3050 50  0001 C CNN "Power"
-F 8 "5%" H 3500 2950 50  0001 C CNN "Tolerance"
-	1    3500 3150
-	0    -1   -1   0
 $EndComp
 $Comp
@@
 	1    0    0    -1
 $EndComp
+$Comp
+L R R3
+U 1 1 530ADB7A
+P 3500 3150
+F 0 "R3" H 3500 3250 50  0000 C CNN
+F 1 "10k" H 3500 3150 50  0000 C CNN
+F 2 "RESC1005-N" H 3500 3150 60  0001 C CNN
+F 3 "~" H 3500 3150 60  0000 C CNN
+F 4 "Yageo" H 3500 3150 60  0001 C CNN "MFR Name"
+F 5 "RC0402FR-0710KL" H 3500 3150 60  0001 C CNN "MFR Part No"
+F 6 "311-10.0KLRCT-ND" H 3500 3150 60  0001 C CNN "Distributor Part No"
+F 7 "1/16W" H 3500 3050 50  0001 C CNN "Power"
+F 8 "1%" H 3500 3050 50  0001 C CNN "Tolerance"
+	1    3500 3150
+	0    -1   -1   0
+$EndComp
 $EndSCHEMATC
