File: Hardware/Transmitter.sch (KiCad schematic (older format))
At the start: 26 parts, among them U2 ADF7012, X1 VCXO

Commit message: Transmitter RF components
Parts:
- C12: value C -> 1200pF; footprint ~ -> CAPC1005-N; Dielectric D -> X7R; Distributor Part No (none) -> 1276-1515-1-ND; MFR Name (none) -> Samsung; MFR Part No (none) -> CL05B122KB5NNNC; Voltage V -> 50V
- C13: value C -> 0.018uF; footprint ~ -> CAPC1005-N; Dielectric D -> X7R; Distributor Part No (none) -> 1276-1527-1-ND; MFR Name (none) -> Samsung; MFR Part No (none) -> CL05B183KA5NNNC; Voltage V -> 25V
- C14: value C -> 560pF; footprint ~ -> CAPC1005-N; Dielectric D -> X7R; Distributor Part No (none) -> 311-1029-1-ND; MFR Name (none) -> Yageo; MFR Part No (none) -> CC0402KRX7R9BB561; Voltage V -> 50V
- C20: value C -> 470pF
- C21, C23: value C -> 3.3pF; footprint ~ -> CAPC1005-N; Dielectric D -> NP0; Distributor Part No (none) -> 1276-1141-1-ND; MFR Name (none) -> Samsung; MFR Part No (none) -> CL05C3R3CB5NNNC; Voltage V -> 50V
- C22: value C -> 8.2pF; footprint ~ -> CAPC1005-N; Dielectric D -> NP0; Distributor Part No (none) -> 1276-1730-1-ND; MFR Name (none) -> Samsung; MFR Part No (none) -> CL05C8R2DB5NNNC; Voltage V -> 50V
- C8: footprint CAPC1608-N -> CAPC1005-N; Dielectric X7R -> D; Distributor Part No 1276-1005-1-ND -> (none); MFR Name Samsung -> (none); MFR Part No CL10B104KO8NNNC -> (none); Voltage 16V -> V
- L3: value L -> 19.2nH; footprint ~ -> INDC1005-N; Distributor Part No (none) -> AISC-0402-19NG-TCT-ND; MFR Name (none) -> Abracon; MFR Part No (none) -> AISC-0402-19NG-T
- L4, L6, L7: value L -> 22nH; footprint ~ -> INDC1005-N; Distributor Part No (none) -> 587-1523-1-ND; MFR Name (none) -> Taiyo Yuden; MFR Part No (none) -> HK100522NJ-T
- L5: value L -> 10pF; footprint ~ -> INDC1005-N; Distributor Part No (none) -> 311-1014-1-ND; MFR Name (none) -> Yageo; MFR Part No (none) -> CC0402JRNPO9BN100
- R5: value R -> 820; footprint ~ -> RESC1005-N; Distributor Part No (none) -> 311-820JRCT-ND; MFR Name (none) -> Yageo; MFR Part No (none) -> RC0402JR-07820RL; Power W -> 1/16W; Tolerance % -> 5%
- R6: value R -> 1.6k; footprint ~ -> RESC1005-N; Distributor Part No (none) -> P1.6KJCT-ND; MFR Name (none) -> Panasonic; MFR Part No (none) -> ERJ-2GEJ162X; Power W -> 1/10W; Tolerance % -> 5%
Changed lines of the file:
@@
 Sheet 3 4
 Title "Aether - Pico Tracker"
-Date "6 feb 2014"
+Date "7 feb 2014"
 Rev "1"
 Comp "Aerodyne Labs"
@@
 P 6200 5750
 F 0 "L3" H 6200 5650 60  0000 C CNN
-F 1 "L" H 6200 5800 60  0000 C CNN
-F 2 "~" H 6200 5750 60  0000 C CNN
+F 1 "19.2nH" H 6200 5800 60  0000 C CNN
+F 2 "INDC1005-N" H 6200 5750 60  0001 C CNN
 F 3 "~" H 6200 5750 60  0000 C CNN
+F 4 "Abracon" H 6200 5750 60  0001 C CNN "MFR Name"
+F 5 "AISC-0402-19NG-T" H 6200 5750 60  0001 C CNN "MFR Part No"
+F 6 "AISC-0402-19NG-TCT-ND" H 6200 5750 60  0001 C CNN "Distributor Part No"
 	1    6200 5750
 	0    -1   -1   0
@@
 P 3900 5750
 F 0 "C12" H 3950 5900 60  0000 L CNN
-F 1 "C" H 3950 5600 60  0000 L CNN
-F 2 "~" H 3900 5750 60  0000 C CNN
+F 1 "1200pF" H 3950 5600 60  0000 L CNN
+F 2 "CAPC1005-N" H 3900 5750 60  0001 C CNN
 F 3 "~" H 3900 5750 60  0000 C CNN
-F 4 "V" H 3850 5600 60  0001 R CNN "Voltage"
-F 5 "D" H 3850 5900 60  0001 R CNN "Dielectric"
+F 4 "Samsung" H 3900 5750 60  0001 C CNN "MFR Name"
+F 5 "CL05B122KB5NNNC" H 3900 5750 60  0001 C CNN "MFR Part No"
+F 6 "1276-1515-1-ND" H 3900 5750 60  0001 C CNN "Distributor Part No"
+F 7 "50V" H 3850 5600 60  0001 R CNN "Voltage"
+F 8 "X7R" H 3850 5900 60  0001 R CNN "Dielectric"
 	1    3900 5750
-	1    0    0    -1
+	-1   0    0    -1
 $EndComp
 $Comp
@@
 P 4300 6350
 F 0 "C13" H 4350 6500 60  0000 L CNN
-F 1 "C" H 4350 6200 60  0000 L CNN
-F 2 "~" H 4300 6350 60  0000 C CNN
+F 1 "0.018uF" H 4350 6200 60  0000 L CNN
+F 2 "CAPC1005-N" H 4300 6350 60  0001 C CNN
 F 3 "~" H 4300 6350 60  0000 C CNN
-F 4 "V" H 4250 6200 60  0001 R CNN "Voltage"
-F 5 "D" H 4250 6500 60  0001 R CNN "Dielectric"
+F 4 "Samsung" H 4300 6350 60  0001 C CNN "MFR Name"
+F 5 "CL05B183KA5NNNC" H 4300 6350 60  0001 C CNN "MFR Part No"
+F 6 "1276-1527-1-ND" H 4300 6350 60  0001 C CNN "Distributor Part No"
+F 7 "25V" H 4250 6200 60  0001 R CNN "Voltage"
+F 8 "X7R" H 4250 6500 60  0001 R CNN "Dielectric"
 	1    4300 6350
 	1    0    0    -1
@@
 P 4300 5750
 F 0 "R5" H 4300 5850 50  0000 C CNN
-F 1 "R" H 4300 5750 50  0000 C CNN
-F 2 "~" H 4300 5750 60  0000 C CNN
+F 1 "820" H 4300 5750 50  0000 C CNN
+F 2 "RESC1005-N" H 4300 5750 60  0001 C CNN
 F 3 "~" H 4300 5750 60  0000 C CNN
-F 4 "W" H 4300 5650 50  0001 C CNN "Power"
-F 5 "%" H 4300 5550 50  0001 C CNN "Tolerance"
+F 4 "Yageo" H 4300 5750 60  0001 C CNN "MFR Name"
+F 5 "RC0402JR-07820RL" H 4300 5750 60  0001 C CNN "MFR Part No"
+F 6 "311-820JRCT-ND" H 4300 5750 60  0001 C CNN "Distributor Part No"
+F 7 "1/16W" H 4300 5650 50  0001 C CNN "Power"
+F 8 "5%" H 4300 5550 50  0001 C CNN "Tolerance"
 	1    4300 5750
 	0    -1   -1   0
@@
 P 4750 5400
 F 0 "R6" H 4750 5500 50  0000 C CNN
-F 1 "R" H 4750 5400 50  0000 C CNN
-F 2 "~" H 4750 5400 60  0000 C CNN
+F 1 "1.6k" H 4750 5400 50  0000 C CNN
+F 2 "RESC1005-N" H 4750 5400 60  0001 C CNN
 F 3 "~" H 4750 5400 60  0000 C CNN
-F 4 "W" H 4750 5300 50  0001 C CNN "Power"
-F 5 "%" H 4750 5200 50  0001 C CNN "Tolerance"
+F 4 "Panasonic" H 4750 5400 60  0001 C CNN "MFR Name"
+F 5 "ERJ-2GEJ162X" H 4750 5400 60  0001 C CNN "MFR Part No"
+F 6 "P1.6KJCT-ND" H 4750 5400 60  0001 C CNN "Distributor Part No"
+F 7 "1/10W" H 4750 5300 50  0001 C CNN "Power"
+F 8 "5%" H 4750 5200 50  0001 C CNN "Tolerance"
 	1    4750 5400
 	1    0    0    -1
@@
 P 5200 5750
 F 0 "C14" H 5250 5900 60  0000 L CNN
-F 1 "C" H 5250 5600 60  0000 L CNN
-F 2 "~" H 5200 5750 60  0000 C CNN
+F 1 "560pF" H 5250 5600 60  0000 L CNN
+F 2 "CAPC1005-N" H 5200 5750 60  0001 C CNN
 F 3 "~" H 5200 5750 60  0000 C CNN
-F 4 "V" H 5150 5600 60  0001 R CNN "Voltage"
-F 5 "D" H 5150 5900 60  0001 R CNN "Dielectric"
+F 4 "Yageo" H 5200 5750 60  0001 C CNN "MFR Name"
+F 5 "CC0402KRX7R9BB561" H 5200 5750 60  0001 C CNN "MFR Part No"
+F 6 "311-1029-1-ND" H 5200 5750 60  0001 C CNN "Distributor Part No"
+F 7 "50V" H 5150 5600 60  0001 R CNN "Voltage"
+F 8 "X7R" H 5150 5900 60  0001 R CNN "Dielectric"
 	1    5200 5750
 	1    0    0    -1
@@
 RFGnd
 $Comp
-L L L4
-U 1 1 52ECC2CB
-P 7100 5250
-F 0 "L4" H 7100 5150 60  0000 C CNN
-F 1 "L" H 7100 5300 60  0000 C CNN
-F 2 "~" H 7100 5250 60  0000 C CNN
-F 3 "~" H 7100 5250 60  0000 C CNN
-	1    7100 5250
-	0    -1   -1   0
-$EndComp
-$Comp
-L L L5
-U 1 1 52ECC2DA
-P 7550 5700
-F 0 "L5" H 7550 5600 60  0000 C CNN
-F 1 "L" H 7550 5750 60  0000 C CNN
-F 2 "~" H 7550 5700 60  0000 C CNN
-F 3 "~" H 7550 5700 60  0000 C CNN
-	1    7550 5700
-	1    0    0    -1
-$EndComp
-$Comp
 L C C20
 U 1 1 52ECC2E9
 P 8250 5700
 F 0 "C20" H 8300 5850 60  0000 L CNN
-F 1 "C" H 8300 5550 60  0000 L CNN
+F 1 "470pF" H 8300 5550 60  0000 L CNN
 F 2 "~" H 8250 5700 60  0000 C CNN
 F 3 "~" H 8250 5700 60  0000 C CNN
@@
 P 8700 6150
 F 0 "C21" H 8750 6300 60  0000 L CNN
-F 1 "C" H 8750 6000 60  0000 L CNN
-F 2 "~" H 8700 6150 60  0000 C CNN
+F 1 "3.3pF" H 8750 6000 60  0000 L CNN
+F 2 "CAPC1005-N" H 8700 6150 60  0001 C CNN
 F 3 "~" H 8700 6150 60  0000 C CNN
-F 4 "V" H 8650 6000 60  0001 R CNN "Voltage"
-F 5 "D" H 8650 6300 60  0001 R CNN "Dielectric"
+F 4 "Samsung" H 8700 6150 60  0001 C CNN "MFR Name"
+F 5 "CL05C3R3CB5NNNC" H 8700 6150 60  0001 C CNN "MFR Part No"
+F 6 "1276-1141-1-ND" H 8700 6150 60  0001 C CNN "Distributor Part No"
+F 7 "50V" H 8650 6000 60  0001 R CNN "Voltage"
+F 8 "NP0" H 8650 6300 60  0001 R CNN "Dielectric"
 	1    8700 6150
 	1    0    0    -1
@@
 P 9150 5700
 F 0 "L6" H 9150 5600 60  0000 C CNN
-F 1 "L" H 9150 5750 60  0000 C CNN
-F 2 "~" H 9150 5700 60  0000 C CNN
+F 1 "22nH" H 9150 5750 60  0000 C CNN
+F 2 "INDC1005-N" H 9150 5700 60  0001 C CNN
 F 3 "~" H 9150 5700 60  0000 C CNN
+F 4 "Taiyo Yuden" H 9150 5700 60  0001 C CNN "MFR Name"
+F 5 "HK100522NJ-T" H 9150 5700 60  0001 C CNN "MFR Part No"
+F 6 "587-1523-1-ND" H 9150 5700 60  0001 C CNN "Distributor Part No"
 	1    9150 5700
-	1    0    0    -1
-$EndComp
-$Comp
-L L L7
-U 1 1 52ECC32E
-P 10050 5700
-F 0 "L7" H 10050 5600 60  0000 C CNN
-F 1 "L" H 10050 5750 60  0000 C CNN
-F 2 "~" H 10050 5700 60  0000 C CNN
-F 3 "~" H 10050 5700 60  0000 C CNN
-	1    10050 5700
 	1    0    0    -1
 $EndComp
@@
 P 9600 6150
 F 0 "C22" H 9650 6300 60  0000 L CNN
-F 1 "C" H 9650 6000 60  0000 L CNN
-F 2 "~" H 9600 6150 60  0000 C CNN
+F 1 "8.2pF" H 9650 6000 60  0000 L CNN
+F 2 "CAPC1005-N" H 9600 6150 60  0001 C CNN
 F 3 "~" H 9600 6150 60  0000 C CNN
-F 4 "V" H 9550 6000 60  0001 R CNN "Voltage"
-F 5 "D" H 9550 6300 60  0001 R CNN "Dielectric"
+F 4 "Samsung" H 9600 6150 60  0001 C CNN "MFR Name"
+F 5 "CL05C8R2DB5NNNC" H 9600 6150 60  0001 C CNN "MFR Part No"
+F 6 "1276-1730-1-ND" H 9600 6150 60  0001 C CNN "Distributor Part No"
+F 7 "50V" H 9550 6000 60  0001 R CNN "Voltage"
+F 8 "NP0" H 9550 6300 60  0001 R CNN "Dielectric"
 	1    9600 6150
-	1    0    0    -1
-$EndComp
-$Comp
-L C C23
-U 1 1 52ECC358
-P 10500 6150
-F 0 "C23" H 10550 6300 60  0000 L CNN
-F 1 "C" H 10550 6000 60  0000 L CNN
-F 2 "~" H 10500 6150 60  0000 C CNN
-F 3 "~" H 10500 6150 60  0000 C CNN
-F 4 "V" H 10450 6000 60  0001 R CNN "Voltage"
-F 5 "D" H 10450 6300 60  0001 R CNN "Dielectric"
-	1    10500 6150
 	1    0    0    -1
 $EndComp
@@
 F 0 "C8" H 1150 4000 60  0000 L CNN
 F 1 "0.1uF" H 1150 3700 60  0000 L CNN
-F 2 "CAPC1608-N" H 1100 3850 60  0001 C CNN
+F 2 "CAPC1005-N" H 1100 3850 60  0001 C CNN
 F 3 "~" H 1100 3850 60  0000 C CNN
-F 4 "Samsung" H 1100 3850 60  0001 C CNN "MFR Name"
-F 5 "CL10B104KO8NNNC" H 1100 3850 60  0001 C CNN "MFR Part No"
-F 6 "1276-1005-1-ND" H 1100 3850 60  0001 C CNN "Distributor Part No"
-F 7 "16V" H 1050 3700 60  0001 R CNN "Voltage"
-F 8 "X7R" H 1050 4000 60  0001 R CNN "Dielectric"
+F 4 "V" H 1050 3700 60  0001 R CNN "Voltage"
+F 5 "D" H 1050 4000 60  0001 R CNN "Dielectric"
 	1    1100 3850
 	1    0    0    -1
@@
 Wire Wire Line
 	2500 3300 2400 3300
+$Comp
+L L L7
+U 1 1 52F55E68
+P 10050 5700
+F 0 "L7" H 10050 5600 60  0000 C CNN
+F 1 "22nH" H 10050 5750 60  0000 C CNN
+F 2 "INDC1005-N" H 10050 5700 60  0001 C CNN
+F 3 "~" H 10050 5700 60  0000 C CNN
+F 4 "Taiyo Yuden" H 10050 5700 60  0001 C CNN "MFR Name"
+F 5 "HK100522NJ-T" H 10050 5700 60  0001 C CNN "MFR Part No"
+F 6 "587-1523-1-ND" H 10050 5700 60  0001 C CNN "Distributor Part No"
+	1    10050 5700
+	1    0    0    -1
+$EndComp
+$Comp
+L L L4
+U 1 1 52F55EAC
+P 7100 5250
+F 0 "L4" H 7100 5150 60  0000 C CNN
+F 1 "22nH" H 7100 5300 60  0000 C CNN
+F 2 "INDC1005-N" H 7100 5250 60  0001 C CNN
+F 3 "~" H 7100 5250 60  0000 C CNN
+F 4 "Taiyo Yuden" H 7100 5250 60  0001 C CNN "MFR Name"
+F 5 "HK100522NJ-T" H 7100 5250 60  0001 C CNN "MFR Part No"
+F 6 "587-1523-1-ND" H 7100 5250 60  0001 C CNN "Distributor Part No"
+	1    7100 5250
+	0    -1   -1   0
+$EndComp
+$Comp
+L L L5
+U 1 1 52ECC2DA
+P 7550 5700
+F 0 "L5" H 7550 5600 60  0000 C CNN
+F 1 "10pF" H 7550 5750 60  0000 C CNN
+F 2 "INDC1005-N" H 7550 5700 60  0001 C CNN
+F 3 "~" H 7550 5700 60  0000 C CNN
+F 4 "Yageo" H 7550 5700 60  0001 C CNN "MFR Name"
+F 5 "CC0402JRNPO9BN100" H 7550 5700 60  0001 C CNN "MFR Part No"
+F 6 "311-1014-1-ND" H 7550 5700 60  0001 C CNN "Distributor Part No"
+	1    7550 5700
+	1    0    0    -1
+$EndComp
+$Comp
+L C C23
+U 1 1 52F56298
+P 10500 6150
+F 0 "C23" H 10550 6300 60  0000 L CNN
+F 1 "3.3pF" H 10550 6000 60  0000 L CNN
+F 2 "CAPC1005-N" H 10500 6150 60  0001 C CNN
+F 3 "~" H 10500 6150 60  0000 C CNN
+F 4 "Samsung" H 10500 6150 60  0001 C CNN "MFR Name"
+F 5 "CL05C3R3CB5NNNC" H 10500 6150 60  0001 C CNN "MFR Part No"
+F 6 "1276-1141-1-ND" H 10500 6150 60  0001 C CNN "Distributor Part No"
+F 7 "50V" H 10450 6000 60  0001 R CNN "Voltage"
+F 8 "NP0" H 10450 6300 60  0001 R CNN "Dielectric"
+	1    10500 6150
+	1    0    0    -1
+$EndComp
 $EndSCHEMATC
