File: Hardware/Transmitter.sch (KiCad schematic (older format))
At the start: 0 parts

Commit message: Add Si4463
Parts:
- added U?: SI446X, symbol SI446X
Changed lines of the file:
@@
 $Descr A4 11693 8268
 encoding utf-8
-Sheet 2 4
+Sheet 4 4
 Title "Aether - Pico Tracker"
 Date "30 jul 2014"
@@
 Comment4 ""
 $EndDescr
+$Comp
+L SI446X U?
+U 1 1 53D877EF
+P 5550 3350
+F 0 "U?" H 5550 3900 60  0000 C CNN
+F 1 "SI446X" H 5550 2800 60  0000 C CNN
+F 2 "" H 5550 3350 60  0000 C CNN
+F 3 "" H 5550 3350 60  0000 C CNN
+	1    5550 3350
+	1    0    0    -1
+$EndComp
+Text HLabel 4700 3100 0    60   Input ~ 0
+SCLK
+Text HLabel 4700 3200 0    60   Output ~ 0
+MISO
+Text HLabel 4700 3300 0    60   Input ~ 0
+MOSI
+Text HLabel 4700 3400 0    60   Input ~ 0
+CS
+Text HLabel 8300 2900 2    60   UnSpc ~ 0
+RF
+Text HLabel 8300 3000 2    60   UnSpc ~ 0
+RFGnd
 $EndSCHEMATC
