File: Hardware/Power.sch (KiCad schematic (older format))
At the start: 15 parts

Commit message: System 3v3 regulator
Parts:
- added C? (x2): C, ~, symbol C
- added D?: DIODE-SCH, ~, symbol DIODE-SCH
- added J?: PWR, ~, symbol CONN-2
- added L?: L, ~, symbol L
- added U?: TPS62203, symbol TPS6220X
- J?: value JUMPER-NO -> BATT
Connections:
- net labels added: +3.3V, STAT1, STAT2, ~PG
- wire segments 52 -> 98
Other:
- moved on the sheet: B?, C?, J?, R?, U?
