File: Hardware/Power.sch (KiCad schematic (older format))
At the start: 14 parts

Commit message: Charger circuitry values
#26
Parts:
- removed RT?: 10k, symbol Thermistor
- added RT?: 10k, symbol Thermistor
- C? (x3): value 10uF -> 4.7uF
- R? (x2): value Resistor -> 100k
- R?: value Resistor -> 2k
- R?: value Resistor -> 36k
Connections:
- net GND: now also RT?.2
- net CHG_EN: now reaches U?.17 (CE)
- net at C?.1, R?.1, U?.18 (IN)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: now also U?.3 (SEL), U?.4 (PROG2), U?.9 (~TE)
- net ~CHG_PG: now reaches U?.6 (~PG)
- net CHG_STAT2: now reaches U?.7 (STAT2)
- net CHG_STAT1: now reaches U?.8 (STAT1)
- net at R?.1, R?.2: now also RT?.1
- net Sense renamed BSense
Changed lines of the file:
@@
 P 8400 3050
 F 0 "C?" V 8250 3150 60  0000 L CNN
-F 1 "10uF" V 8350 3150 60  0000 L CNN
+F 1 "4.7uF" V 8350 3150 60  0000 L CNN
 F 2 "" H 8300 3050 60  0001 C CNN
 F 3 "" H 8400 3150 60  0001 C CNN
@@
 $EndComp
 Wire Wire Line
-	5400 2700 5500 2700
-Wire Wire Line
-	5500 2700 8400 2700
-Wire Wire Line
-	8400 2700 8700 2700
-Wire Wire Line
-	8700 2700 9200 2700
+	5400 2700 9200 2700
 Wire Wire Line
 	8700 2700 8700 2800
@@
 	5400 2800 5500 2800
 Wire Wire Line
-	5500 2700 5500 2800
-Wire Wire Line
-	5500 2800 5500 2900
+	5500 2700 5500 2900
 Connection ~ 5500 2700
 Wire Wire Line
@@
 P 9900 2850
 F 0 "C?" V 9750 2950 60  0000 L CNN
-F 1 "10uF" V 9850 2950 60  0000 L CNN
+F 1 "4.7uF" V 9850 2950 60  0000 L CNN
 F 2 "" H 9800 2850 60  0001 C CNN
 F 3 "" H 9900 2950 60  0001 C CNN
@@
 $EndComp
 Wire Wire Line
-	5400 2500 5500 2500
-Wire Wire Line
-	5500 2500 9900 2500
-Wire Wire Line
-	9900 2400 9900 2500
-Wire Wire Line
-	9900 2500 9900 2600
+	5400 2500 9900 2500
+Wire Wire Line
+	9900 2400 9900 2600
 Wire Wire Line
 	5400 2600 5500 2600
@@
 $EndComp
 Wire Wire Line
-	5500 3400 5500 3500
-Wire Wire Line
-	5500 3500 5500 3600
-Wire Wire Line
-	5500 3600 5500 3700
+	5500 3400 5500 3700
 Wire Wire Line
 	5500 3400 5400 3400
@@
 P 6000 3550
 F 0 "R?" V 5850 3650 60  0000 L CNN
-F 1 "Resistor" V 5950 3650 60  0000 L CNN
+F 1 "100k" V 5950 3650 60  0000 L CNN
 F 2 "" H 5900 3550 60  0001 C CNN
 F 3 "" H 6000 3650 60  0001 C CNN
@@
 P 6300 3550
 F 0 "R?" V 6150 3650 60  0000 L CNN
-F 1 "Resistor" V 6250 3650 60  0000 L CNN
+F 1 "2k" V 6250 3650 60  0000 L CNN
 F 2 "" H 6200 3550 60  0001 C CNN
 F 3 "" H 6300 3650 60  0001 C CNN
@@
 	0    1    1    0
 $EndComp
-$Comp
-L Thermistor RT?
-U 1 1 54996324
-P 7800 3350
-F 0 "RT?" V 7650 3450 60  0000 L CNN
-F 1 "10k" V 7750 3450 60  0000 L CNN
-F 2 "" H 7700 3350 60  0001 C CNN
-F 3 "" H 7800 3450 60  0001 C CNN
-F 4 "Value" H 7800 3350 60  0001 C CNN "Manufacturer"
-F 5 "Value" H 7800 3350 60  0001 C CNN "Manufacturer Part #"
-F 6 "Value" H 7800 3350 60  0001 C CNN "Vendor"
-F 7 "Value" H 7800 3350 60  0001 C CNN "Vendor Part #"
-	1    7800 3350
-	0    1    1    0
-$EndComp
 Wire Wire Line
 	5400 3000 6700 3000
 Wire Wire Line
-	7200 3000 7300 3000
-Wire Wire Line
-	7300 3000 7800 3000
+	7200 3000 7800 3000
 Wire Wire Line
 	7800 3000 7800 3100
@@
 P 3850 1600
 F 0 "C?" V 3700 1700 60  0000 L CNN
-F 1 "10uF" V 3800 1700 60  0000 L CNN
+F 1 "4.7uF" V 3800 1700 60  0000 L CNN
 F 2 "" H 3750 1600 60  0001 C CNN
 F 3 "" H 3850 1700 60  0001 C CNN
@@
 $EndComp
 Wire Wire Line
-	4100 2100 4200 2100
-Wire Wire Line
-	4200 2100 4300 2100
+	4100 2100 4300 2100
 Wire Wire Line
 	4200 2100 4200 2800
@@
 	3600 1600 3500 1600
 Wire Wire Line
-	3500 1600 3500 2100
-Wire Wire Line
-	3500 2100 3500 2500
+	3500 1600 3500 2500
 Wire Wire Line
 	3500 2100 3600 2100
 Wire Wire Line
-	3500 2500 4100 2500
-Wire Wire Line
-	4100 2500 4300 2500
+	3500 2500 4300 2500
 Connection ~ 3500 2100
 Wire Wire Line
 	4300 2600 4100 2600
 Wire Wire Line
-	4100 2600 4100 2500
+	4100 2500 4100 3200
 Connection ~ 4100 2500
 $Comp
@@
 P 9200 3050
 F 0 "R?" V 9050 3150 60  0000 L CNN
-F 1 "Resistor" V 9150 3150 60  0000 L CNN
+F 1 "36k" V 9150 3150 60  0000 L CNN
 F 2 "" H 9100 3050 60  0001 C CNN
 F 3 "" H 9200 3150 60  0001 C CNN
@@
 P 9200 3750
 F 0 "R?" V 9050 3850 60  0000 L CNN
-F 1 "Resistor" V 9150 3850 60  0000 L CNN
+F 1 "100k" V 9150 3850 60  0000 L CNN
 F 2 "" H 9100 3750 60  0001 C CNN
 F 3 "" H 9200 3850 60  0001 C CNN
@@
 	9200 4100 9200 4000
 Text HLabel 9300 3400 2    60   Output ~ 0
-Sense
-Wire Wire Line
-	9200 3300 9200 3400
-Wire Wire Line
-	9200 3400 9200 3500
+BSense
+Wire Wire Line
+	9200 3300 9200 3500
 Wire Wire Line
 	9300 3400 9200 3400
@@
 	9200 2700 9200 2800
 Connection ~ 8700 2700
+Wire Wire Line
+	4100 3100 4300 3100
+Connection ~ 4100 2600
+Wire Wire Line
+	4100 3200 4300 3200
+Connection ~ 4100 3100
+Text HLabel 4000 3400 0    60   Output ~ 0
+~CHG_PG
+Text HLabel 4000 3600 0    60   Output ~ 0
+CHG_STAT1
+Text HLabel 4000 3500 0    60   Output ~ 0
+CHG_STAT2
+Wire Wire Line
+	4000 3400 4300 3400
+Wire Wire Line
+	4300 3500 4000 3500
+Wire Wire Line
+	4000 3600 4300 3600
+$Comp
+L Thermistor RT?
+U 1 1 5499EE33
+P 7800 3350
+F 0 "RT?" V 7650 3450 60  0000 L CNN
+F 1 "10k" V 7750 3450 60  0000 L CNN
+F 2 "" H 7700 3350 60  0001 C CNN
+F 3 "" H 7800 3450 60  0001 C CNN
+F 4 "Murata" H 7800 3350 60  0001 C CNN "Manufacturer"
+F 5 "NCP18XH103J03RB" H 7800 3350 60  0001 C CNN "Manufacturer Part #"
+F 6 "Digikey" H 7800 3350 60  0001 C CNN "Vendor"
+F 7 "490-2436-1-ND" H 7800 3350 60  0001 C CNN "Vendor Part #"
+F 8 "3380k" V 7850 3450 60  0000 L CNN "Sensitivity"
+	1    7800 3350
+	0    1    1    0
+$EndComp
+Wire Wire Line
+	4300 3000 4100 3000
+Connection ~ 4100 3000
+Text HLabel 4000 2900 0    60   Input ~ 0
+CHG_EN
+Wire Wire Line
+	4000 2900 4300 2900
 $EndSCHEMATC

Commit message: Add solar charging capability
Parts:
- added C?: Capacitor, symbol Capacitor
- added D?: Diode-Schottky, symbol Diode-Schottky
- added J?: Solar+, symbol Conn-1
- added J?: Solar-, symbol Conn-1
- added J? (x2): Conn-1, symbol Conn-1
- added R?: Resistor, symbol Resistor
- added R?: 100k, symbol Resistor
Connections:
- net GND: now also C?.2, J?.1, J?.1, R?.2
- net +5VP: now reaches C?.1, R?.1, U?.18 (IN), U?.19 (IN), U?.3 (SEL), U?.4 (PROG2), U?.9 (~TE)
- net +5VP: now also C?.1, D?.C
- new net: D?.A, J?.1, J?.1, R?.1
- new net SSense: R?.1, R?.2
Other:
- moved on the sheet: B?, C?, R?, RT?, U?

Commit message: Add 3v3 regulator
Parts:
- added C?: 18pF, symbol Capacitor
- added C?: 10uF, symbol Capacitor
- added C?: 4.7uF, symbol Capacitor
- added L?: 2.2uH, symbol Inductor
- added R?: 453k, symbol Resistor
- added R?: 100k, symbol Resistor
- added U?: NCP1521, symbol NCP1521
- R?: value Resistor -> 100k
Connections:
- net +BATT: now also C?.1, U?.1 (VIN)
- net GND: now also C?.2, C?.2, R?.2, U?.2 (GND)
- new net: C?.2, R?.1, R?.2, U?.4 (FB)
- new net: L?.1, U?.5 (LX)
- new net +3V3: C?.1, C?.1, L?.2, R?.1
Changed lines of the file:
@@
 LIBS:Connectors
 LIBS:Microchip
+LIBS:ONSemiconductor
 LIBS:Aether-cache
 EELAYER 25 0
@@
 P 2100 2650
 F 0 "R?" V 1950 2750 60  0000 L CNN
-F 1 "Resistor" V 2050 2750 60  0000 L CNN
+F 1 "100k" V 2050 2750 60  0000 L CNN
 F 2 "" H 2000 2650 60  0001 C CNN
 F 3 "" H 2100 2750 60  0001 C CNN
@@
 	2000 3000 2100 3000
 Connection ~ 2100 3000
+$Comp
+L NCP1521 U?
+U 1 1 549A4164
+P 3400 5550
+F 0 "U?" H 3400 6000 60  0000 C CNN
+F 1 "NCP1521" H 3400 5100 60  0000 C CNN
+F 2 "" H 3400 5550 60  0000 C CNN
+F 3 "" H 3400 5550 60  0000 C CNN
+F 4 "Value" H 3400 5550 60  0001 C CNN "ON Semi"
+F 5 "NCP1521BSNT1G" H 3400 5550 60  0001 C CNN "Manufacturer Part #"
+F 6 "Digikey" H 3400 5550 60  0001 C CNN "Vendor"
+F 7 "NCP1521BSNT1GOSCT-ND" H 3400 5550 60  0001 C CNN "Vendor Part #"
+	1    3400 5550
+	1    0    0    -1
+$EndComp
+$Comp
+L Inductor L?
+U 1 1 549A41CA
+P 4150 5200
+F 0 "L?" V 4000 5300 60  0000 L CNN
+F 1 "2.2uH" V 4100 5300 60  0000 L CNN
+F 2 "" H 4050 5200 60  0001 C CNN
+F 3 "" H 4150 5300 60  0001 C CNN
+F 4 "Value" H 4150 5200 60  0001 C CNN "Manufacturer"
+F 5 "Value" H 4150 5200 60  0001 C CNN "Manufacturer Part #"
+F 6 "Value" H 4150 5200 60  0001 C CNN "Vendor"
+F 7 "Value" H 4150 5200 60  0001 C CNN "Vendor Part #"
+F 8 "0.25A" V 4200 5300 50  0000 L CNN "Current"
+F 9 "100mO" V 4300 5300 50  0000 L CNN "DCR"
+	1    4150 5200
+	1    0    0    -1
+$EndComp
+$Comp
+L Resistor R?
+U 1 1 549A422F
+P 4500 5550
+F 0 "R?" V 4350 5650 60  0000 L CNN
+F 1 "453k" V 4450 5650 60  0000 L CNN
+F 2 "" H 4400 5550 60  0001 C CNN
+F 3 "" H 4500 5650 60  0001 C CNN
+F 4 "Value" H 4500 5550 60  0001 C CNN "Manufacturer"
+F 5 "Value" H 4500 5550 60  0001 C CNN "Manufacturer Part #"
+F 6 "Value" H 4500 5550 60  0001 C CNN "Vendor"
+F 7 "Value" H 4500 5550 60  0001 C CNN "Vendor Part #"
+F 8 "1/10W" V 4550 5650 50  0000 L CNN "Power"
+F 9 "5%" V 4650 5650 50  0000 L CNN "Tolerance"
+	1    4500 5550
+	0    -1   1    0
+$EndComp
+$Comp
+L Resistor R?
+U 1 1 549A4298
+P 4500 6250
+F 0 "R?" V 4350 6350 60  0000 L CNN
+F 1 "100k" V 4450 6350 60  0000 L CNN
+F 2 "" H 4400 6250 60  0001 C CNN
+F 3 "" H 4500 6350 60  0001 C CNN
+F 4 "Value" H 4500 6250 60  0001 C CNN "Manufacturer"
+F 5 "Value" H 4500 6250 60  0001 C CNN "Manufacturer Part #"
+F 6 "Value" H 4500 6250 60  0001 C CNN "Vendor"
+F 7 "Value" H 4500 6250 60  0001 C CNN "Vendor Part #"
+F 8 "1/10W" V 4550 6350 50  0000 L CNN "Power"
+F 9 "5%" V 4650 6350 50  0000 L CNN "Tolerance"
+	1    4500 6250
+	0    -1   1    0
+$EndComp
+$Comp
+L Capacitor C?
+U 1 1 549A42EF
+P 4800 5550
+F 0 "C?" V 4650 5650 60  0000 L CNN
+F 1 "18pF" V 4750 5650 60  0000 L CNN
+F 2 "" H 4700 5550 60  0001 C CNN
+F 3 "" H 4800 5650 60  0001 C CNN
+F 4 "Value" H 4800 5550 60  0001 C CNN "Manufacturer"
+F 5 "Value" H 4800 5550 60  0001 C CNN "Manufacturer Part #"
+F 6 "Value" H 4800 5550 60  0001 C CNN "Vendor"
+F 7 "Value" H 4800 5550 60  0001 C CNN "Vendor Part #"
+F 8 "10V" V 4850 5650 50  0000 L CNN "Voltage"
+F 9 "X5R" V 4950 5650 50  0000 L CNN "Dielectric"
+	1    4800 5550
+	0    1    1    0
+$EndComp
+$Comp
+L Capacitor C?
+U 1 1 549A4356
+P 5500 5550
+F 0 "C?" V 5350 5650 60  0000 L CNN
+F 1 "10uF" V 5450 5650 60  0000 L CNN
+F 2 "" H 5400 5550 60  0001 C CNN
+F 3 "" H 5500 5650 60  0001 C CNN
+F 4 "Value" H 5500 5550 60  0001 C CNN "Manufacturer"
+F 5 "Value" H 5500 5550 60  0001 C CNN "Manufacturer Part #"
+F 6 "Value" H 5500 5550 60  0001 C CNN "Vendor"
+F 7 "Value" H 5500 5550 60  0001 C CNN "Vendor Part #"
+F 8 "10V" V 5550 5650 50  0000 L CNN "Voltage"
+F 9 "X5R" V 5650 5650 50  0000 L CNN "Dielectric"
+	1    5500 5550
+	0    1    1    0
+$EndComp
+$Comp
+L +3V3 #PWR?
+U 1 1 549A4420
+P 5500 5100
+F 0 "#PWR?" H 5500 4950 60  0001 C CNN
+F 1 "+3V3" H 5500 5240 60  0000 C CNN
+F 2 "" H 5500 5100 60  0000 C CNN
+F 3 "" H 5500 5100 60  0000 C CNN
+	1    5500 5100
+	1    0    0    -1
+$EndComp
+Wire Wire Line
+	5500 5100 5500 5300
+$Comp
+L GND #PWR?
+U 1 1 549A44A6
+P 4500 6600
+F 0 "#PWR?" H 4500 6350 60  0001 C CNN
+F 1 "GND" H 4500 6450 60  0000 C CNN
+F 2 "" H 4500 6600 60  0000 C CNN
+F 3 "" H 4500 6600 60  0000 C CNN
+	1    4500 6600
+	1    0    0    -1
+$EndComp
+$Comp
+L GND #PWR?
+U 1 1 549A44BA
+P 5500 5900
+F 0 "#PWR?" H 5500 5650 60  0001 C CNN
+F 1 "GND" H 5500 5750 60  0000 C CNN
+F 2 "" H 5500 5900 60  0000 C CNN
+F 3 "" H 5500 5900 60  0000 C CNN
+	1    5500 5900
+	1    0    0    -1
+$EndComp
+Wire Wire Line
+	5500 5900 5500 5800
+Wire Wire Line
+	3800 5200 3900 5200
+Wire Wire Line
+	4400 5200 5500 5200
+Connection ~ 5500 5200
+Wire Wire Line
+	4500 5300 4500 5200
+Connection ~ 4500 5200
+Wire Wire Line
+	4500 5800 4500 6000
+Wire Wire Line
+	4500 6500 4500 6600
+Wire Wire Line
+	4800 5900 4800 5800
+Wire Wire Line
+	3800 5900 4800 5900
+Connection ~ 4500 5900
+Wire Wire Line
+	4800 5300 4800 5200
+Connection ~ 4800 5200
+$Comp
+L Capacitor C?
+U 1 1 549A4AF8
+P 2400 5550
+F 0 "C?" V 2250 5650 60  0000 L CNN
+F 1 "4.7uF" V 2350 5650 60  0000 L CNN
+F 2 "" H 2300 5550 60  0001 C CNN
+F 3 "" H 2400 5650 60  0001 C CNN
+F 4 "Value" H 2400 5550 60  0001 C CNN "Manufacturer"
+F 5 "Value" H 2400 5550 60  0001 C CNN "Manufacturer Part #"
+F 6 "Value" H 2400 5550 60  0001 C CNN "Vendor"
+F 7 "Value" H 2400 5550 60  0001 C CNN "Vendor Part #"
+F 8 "10V" V 2450 5650 50  0000 L CNN "Voltage"
+F 9 "X5R" V 2550 5650 50  0000 L CNN "Dielectric"
+	1    2400 5550
+	0    -1   1    0
+$EndComp
+$Comp
+L +BATT #PWR?
+U 1 1 549A4C75
+P 2400 5100
+F 0 "#PWR?" H 2400 4950 60  0001 C CNN
+F 1 "+BATT" H 2400 5240 60  0000 C CNN
+F 2 "" H 2400 5100 60  0000 C CNN
+F 3 "" H 2400 5100 60  0000 C CNN
+	1    2400 5100
+	1    0    0    -1
+$EndComp
+Wire Wire Line
+	2400 5100 2400 5300
+Wire Wire Line
+	3000 5200 2400 5200
+Connection ~ 2400 5200
+$Comp
+L GND #PWR?
+U 1 1 549A4D8D
+P 2400 5900
+F 0 "#PWR?" H 2400 5650 60  0001 C CNN
+F 1 "GND" H 2400 5750 60  0000 C CNN
+F 2 "" H 2400 5900 60  0000 C CNN
+F 3 "" H 2400 5900 60  0000 C CNN
+	1    2400 5900
+	1    0    0    -1
+$EndComp
+$Comp
+L GND #PWR?
+U 1 1 549A4DA1
+P 2900 6000
+F 0 "#PWR?" H 2900 5750 60  0001 C CNN
+F 1 "GND" H 2900 5850 60  0000 C CNN
+F 2 "" H 2900 6000 60  0000 C CNN
+F 3 "" H 2900 6000 60  0000 C CNN
+	1    2900 6000
+	1    0    0    -1
+$EndComp
+Wire Wire Line
+	2900 6000 2900 5900
+Wire Wire Line
+	2900 5900 3000 5900
+Wire Wire Line
+	2400 5800 2400 5900
 $EndSCHEMATC

Commit message: Add power switch
Parts:
- added SW?: DPDT, symbol DPDT
Connections:
- net +BATT: now also SW?.3
- net GND: now also SW?.1
- net PWR: now reaches U?.3 (EN)
- net PWR: now also SW?.2
Other:
- moved on the sheet: C?
Changed lines of the file:
@@
 $EndComp
 Wire Wire Line
-	5400 2400 9200 2400
+	5400 2400 5500 2400
+Wire Wire Line
+	5500 2400 8400 2400
+Wire Wire Line
+	8400 2400 8700 2400
+Wire Wire Line
+	8700 2400 9200 2400
 Wire Wire Line
 	8700 2400 8700 2500
@@
 	5400 2500 5500 2500
 Wire Wire Line
-	5500 2400 5500 2600
+	5500 2400 5500 2500
+Wire Wire Line
+	5500 2500 5500 2600
 Connection ~ 5500 2400
 Wire Wire Line
@@
 $EndComp
 Wire Wire Line
-	5400 2200 9900 2200
-Wire Wire Line
-	9900 2100 9900 2300
+	5400 2200 5500 2200
+Wire Wire Line
+	5500 2200 9900 2200
+Wire Wire Line
+	9900 2100 9900 2200
+Wire Wire Line
+	9900 2200 9900 2300
 Wire Wire Line
 	5400 2300 5500 2300
@@
 $EndComp
 Wire Wire Line
-	5500 3100 5500 3400
+	5500 3100 5500 3200
+Wire Wire Line
+	5500 3200 5500 3300
+Wire Wire Line
+	5500 3300 5500 3400
 Wire Wire Line
 	5500 3100 5400 3100
@@
 	5400 2700 6700 2700
 Wire Wire Line
-	7200 2700 7800 2700
+	7200 2700 7300 2700
+Wire Wire Line
+	7300 2700 7800 2700
 Wire Wire Line
 	7800 2700 7800 2800
@@
 $EndComp
 Wire Wire Line
-	4100 1800 4300 1800
+	4100 1800 4200 1800
+Wire Wire Line
+	4200 1800 4300 1800
 Wire Wire Line
 	4200 1800 4200 2500
@@
 	3600 1300 3500 1300
 Wire Wire Line
-	3500 2200 3500 1100
+	3500 2200 3500 1800
+Wire Wire Line
+	3500 1800 3500 1300
+Wire Wire Line
+	3500 1300 3500 1100
 Wire Wire Line
 	3500 1800 3600 1800
 Wire Wire Line
-	2700 2200 4300 2200
+	2700 2200 2800 2200
+Wire Wire Line
+	2800 2200 3500 2200
+Wire Wire Line
+	3500 2200 4100 2200
+Wire Wire Line
+	4100 2200 4300 2200
 Connection ~ 3500 1800
 Wire Wire Line
 	4300 2300 4100 2300
 Wire Wire Line
-	4100 2200 4100 2900
+	4100 2200 4100 2300
+Wire Wire Line
+	4100 2300 4100 2700
+Wire Wire Line
+	4100 2700 4100 2800
+Wire Wire Line
+	4100 2800 4100 2900
 Connection ~ 4100 2200
 $Comp
@@
 BSense
 Wire Wire Line
-	9200 3000 9200 3200
+	9200 3000 9200 3100
+Wire Wire Line
+	9200 3100 9200 3200
 Wire Wire Line
 	9300 3100 9200 3100
@@
 $EndComp
 Wire Wire Line
-	2100 1000 2100 1400
+	2100 1000 2100 1300
+Wire Wire Line
+	2100 1300 2100 1400
 Wire Wire Line
 	2100 1000 2000 1000
 Wire Wire Line
-	2000 2200 2200 2200
+	2000 2200 2100 2200
+Wire Wire Line
+	2100 2200 2200 2200
 $Comp
 L Conn-1 J?
@@
 	2000 1900 2100 1900
 Wire Wire Line
-	2100 1900 2100 2400
+	2100 1900 2100 2200
+Wire Wire Line
+	2100 2200 2100 2400
 Connection ~ 2100 2200
 $Comp
@@
 SSense
 Wire Wire Line
-	2100 2900 2100 3100
+	2100 2900 2100 3000
+Wire Wire Line
+	2100 3000 2100 3100
 Wire Wire Line
 	2000 3000 2100 3000
@@
 $EndComp
 Wire Wire Line
-	5500 5100 5500 5300
+	5500 5100 5500 5200
+Wire Wire Line
+	5500 5200 5500 5300
 $Comp
 L GND #PWR?
@@
 	3800 5200 3900 5200
 Wire Wire Line
-	4400 5200 5500 5200
+	4400 5200 4500 5200
+Wire Wire Line
+	4500 5200 4800 5200
+Wire Wire Line
+	4800 5200 5500 5200
 Connection ~ 5500 5200
 Wire Wire Line
@@
 Connection ~ 4500 5200
 Wire Wire Line
-	4500 5800 4500 6000
+	4500 5800 4500 5900
+Wire Wire Line
+	4500 5900 4500 6000
 Wire Wire Line
 	4500 6500 4500 6600
@@
 	4800 5900 4800 5800
 Wire Wire Line
-	3800 5900 4800 5900
+	3800 5900 4500 5900
+Wire Wire Line
+	4500 5900 4800 5900
 Connection ~ 4500 5900
 Wire Wire Line
@@
 L Capacitor C?
 U 1 1 549A4AF8
-P 2400 5550
-F 0 "C?" V 2250 5650 60  0000 L CNN
-F 1 "4.7uF" V 2350 5650 60  0000 L CNN
-F 2 "" H 2300 5550 60  0001 C CNN
-F 3 "" H 2400 5650 60  0001 C CNN
-F 4 "Value" H 2400 5550 60  0001 C CNN "Manufacturer"
-F 5 "Value" H 2400 5550 60  0001 C CNN "Manufacturer Part #"
-F 6 "Value" H 2400 5550 60  0001 C CNN "Vendor"
-F 7 "Value" H 2400 5550 60  0001 C CNN "Vendor Part #"
-F 8 "10V" V 2450 5650 50  0000 L CNN "Voltage"
-F 9 "X5R" V 2550 5650 50  0000 L CNN "Dielectric"
-	1    2400 5550
+P 2500 5550
+F 0 "C?" V 2350 5650 60  0000 L CNN
+F 1 "4.7uF" V 2450 5650 60  0000 L CNN
+F 2 "" H 2400 5550 60  0001 C CNN
+F 3 "" H 2500 5650 60  0001 C CNN
+F 4 "Value" H 2500 5550 60  0001 C CNN "Manufacturer"
+F 5 "Value" H 2500 5550 60  0001 C CNN "Manufacturer Part #"
+F 6 "Value" H 2500 5550 60  0001 C CNN "Vendor"
+F 7 "Value" H 2500 5550 60  0001 C CNN "Vendor Part #"
+F 8 "10V" V 2550 5650 50  0000 L CNN "Voltage"
+F 9 "X5R" V 2650 5650 50  0000 L CNN "Dielectric"
+	1    2500 5550
 	0    -1   1    0
 $EndComp
@@
 L +BATT #PWR?
 U 1 1 549A4C75
-P 2400 5100
-F 0 "#PWR?" H 2400 4950 60  0001 C CNN
-F 1 "+BATT" H 2400 5240 60  0000 C CNN
-F 2 "" H 2400 5100 60  0000 C CNN
-F 3 "" H 2400 5100 60  0000 C CNN
-	1    2400 5100
-	1    0    0    -1
-$EndComp
-Wire Wire Line
-	2400 5100 2400 5300
-Wire Wire Line
-	3000 5200 2400 5200
-Connection ~ 2400 5200
+P 2500 4900
+F 0 "#PWR?" H 2500 4750 60  0001 C CNN
+F 1 "+BATT" H 2500 5040 60  0000 C CNN
+F 2 "" H 2500 4900 60  0000 C CNN
+F 3 "" H 2500 4900 60  0000 C CNN
+	1    2500 4900
+	1    0    0    -1
+$EndComp
+Wire Wire Line
+	2500 4900 2500 5200
+Wire Wire Line
+	2500 5200 2500 5300
+Wire Wire Line
+	3000 5200 2500 5200
+Connection ~ 2500 5200
 $Comp
 L GND #PWR?
 U 1 1 549A4D8D
-P 2400 5900
-F 0 "#PWR?" H 2400 5650 60  0001 C CNN
-F 1 "GND" H 2400 5750 60  0000 C CNN
-F 2 "" H 2400 5900 60  0000 C CNN
-F 3 "" H 2400 5900 60  0000 C CNN
-	1    2400 5900
+P 2500 5900
+F 0 "#PWR?" H 2500 5650 60  0001 C CNN
+F 1 "GND" H 2500 5750 60  0000 C CNN
+F 2 "" H 2500 5900 60  0000 C CNN
+F 3 "" H 2500 5900 60  0000 C CNN
+	1    2500 5900
 	1    0    0    -1
 $EndComp
@@
 	2900 5900 3000 5900
 Wire Wire Line
-	2400 5800 2400 5900
+	2500 5800 2500 5900
+Wire Wire Line
+	3000 5300 2900 5300
+$Comp
+L DPDT SW?
+U 1 1 549A5C86
+P 1550 5300
+F 0 "SW?" H 1550 5500 60  0000 C CNN
+F 1 "DPDT" H 1550 5100 60  0000 C CNN
+F 2 "" H 1550 5300 60  0000 C CNN
+F 3 "" H 1550 5300 60  0000 C CNN
+	1    1550 5300
+	1    0    0    1
+$EndComp
+Text Label 2900 5300 2    60   ~ 0
+PWR
+Text Label 1200 5300 2    60   ~ 0
+PWR
+$Comp
+L +BATT #PWR?
+U 1 1 549A61C5
+P 1900 5100
+F 0 "#PWR?" H 1900 4950 60  0001 C CNN
+F 1 "+BATT" H 1900 5240 60  0000 C CNN
+F 2 "" H 1900 5100 60  0000 C CNN
+F 3 "" H 1900 5100 60  0000 C CNN
+	1    1900 5100
+	1    0    0    -1
+$EndComp
+Wire Wire Line
+	1900 5100 1900 5200
+Wire Wire Line
+	1900 5200 1800 5200
+$Comp
+L GND #PWR?
+U 1 1 549A629F
+P 1900 5500
+F 0 "#PWR?" H 1900 5250 60  0001 C CNN
+F 1 "GND" H 1900 5350 60  0000 C CNN
+F 2 "" H 1900 5500 60  0000 C CNN
+F 3 "" H 1900 5500 60  0000 C CNN
+	1    1900 5500
+	1    0    0    -1
+$EndComp
+Wire Wire Line
+	1900 5500 1900 5400
+Wire Wire Line
+	1900 5400 1800 5400
+Wire Wire Line
+	1200 5300 1300 5300
 $EndSCHEMATC

Commit message: Oscillator selection
Closes #35
Parts:
- SW?: Manufacturer (none) -> C&K Components; Manufacturer Part # (none) -> JS202011SCQN; Vendor (none) -> Digikey; Vendor Part # (none) -> 401-2002-1-ND
Changed lines of the file:
@@
 F 2 "" H 1550 5300 60  0000 C CNN
 F 3 "" H 1550 5300 60  0000 C CNN
+F 4 "C&K Components" H 1550 5300 60  0001 C CNN "Manufacturer"
+F 5 "JS202011SCQN" H 1550 5300 60  0001 C CNN "Manufacturer Part #"
+F 6 "Digikey" H 1550 5300 60  0001 C CNN "Vendor"
+F 7 "401-2002-1-ND" H 1550 5300 60  0001 C CNN "Vendor Part #"
 	1    1550 5300
 	1    0    0    1

Commit message: Power sheet BOM fields
Remove annotations
Parts:
- removed C? (x3): 4.7uF, symbol Capacitor
- removed R? (x5): 100k, symbol Resistor
- removed R?: 36k, symbol Resistor
- added C29, C34, C35: 4.7uF, symbol Capacitor
- added R10, R13, R14, R15, R20: 100k, symbol Resistor
- added R19: 36k, symbol Resistor
- C31: renamed from C?; Manufacturer Value -> Samsung; Manufacturer Part # Value -> CL21A475KPCLNNC; Vendor Value -> Digikey; Vendor Part # Value -> 1276-2417-1-ND
- C32: renamed from C?; Dielectric X5R -> NP0; Manufacturer Value -> Samsung; Manufacturer Part # Value -> CL10C180JB8NNNC; Vendor Value -> Digikey; Vendor Part # Value -> 1276-1089-1-ND; Voltage 10V -> 50V
- C33: renamed from C?; Manufacturer Value -> Samsung; Manufacturer Part # Value -> CL21A106KPFNNNE; Vendor Value -> Digikey; Vendor Part # Value -> 1276-1052-1-ND
- D3: renamed from D?; value Diode-Schottky -> MBR120ESFT1G; Current I -> 1A; Forward Voltage Vf -> 530mV; Manufacturer Value -> ON Semi; Manufacturer Part # Value -> MBR120ESFT1G; Reverse Voltage Vr -> 20V; Vendor Value -> Digikey; Vendor Part # Value -> MBR120ESFT1GOSCT-ND
- L7: renamed from L?; Current 0.25A -> 650mA; DCR 100mO -> 150mO; Manufacturer Value -> TDK; Manufacturer Part # Value -> MLZ2012A2R2M; Vendor Value -> Digikey; Vendor Part # Value -> 445-3168-1-ND
- R11: renamed from R?; Manufacturer Value -> Yageo; Manufacturer Part # Value -> RC0603JR-07270KL; Vendor Value -> Digikey; Vendor Part # Value -> 311-270KGRCT-ND
- R12: renamed from R?; Manufacturer Value -> Yageo; Manufacturer Part # Value -> RC0603FR-07453KL; Tolerance 5% -> 1%; Vendor Value -> Digikey; Vendor Part # Value -> 311-453KHRCT-ND
- R16: renamed from R?; Manufacturer Value -> Yageo; Manufacturer Part # Value -> RC0603JR-072KL; Vendor Value -> Digikey; Vendor Part # Value -> 311-2.0KGRCT-ND
- R9: renamed from R?; Manufacturer Value -> Yageo; Manufacturer Part # Value -> RC0603JR-07100KL; Vendor Value -> Digikey; Vendor Part # Value -> 311-100KGRCT-ND
- U5: renamed from U?; Manufacturer (none) -> ON Semi; ON Semi Value -> (none)
- U6: renamed from U?; Manufacturer (none) -> Microchip; Manufacturer Part # (none) -> MCP73871-2AAI/ML; Vendor (none) -> Digikey; Vendor Part # (none) -> MCP73871-2AAI/ML-ND
- gave numbers to parts that had none: 10
Connections:
- net +BATT: now also C29.1, C35.1
- net BSense: now also R19.2, R20.1
- net GND: now also C29.2, C34.2, C35.2, R10.2, R13.2, R14.2, R15.2, R20.2
- net SSense: now also R10.1
- net at U6.12 (PROG3): now also R15.1
- net at B1.1, U6.14 (VBAT), U6.15 (VBAT)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: now also C34.1, R19.1
- net at R11.2, U6.2 (VPCC): now also R14.1
- net at C32.2, R12.2, U5.4 (FB): now also R13.1
