File: Hardware/Power.sch (KiCad schematic (older format))
At the start: 30 parts, among them J4 Solar-, J5 Conn-1, J6 Conn-1, J7 Solar+, SW1 DPDT, U5 NCP1521, U6 MCP73871

Commit message: Small changes
Parts:
- B1: footprint (none) -> Batteries:Batt_PL-703562-2C-Folded
- C29, C30, C31, C32, C34, C35: footprint (none) -> Capacitors:CAPC1608N
- C33: footprint (none) -> Capacitors:CAPC2012N
- D3: footprint (none) -> Diodes:SODFL3616N
- L7: footprint (none) -> Inductors:INDC2012N
- R10, R11, R12, R13, R14, R15, R16, R17, R18, R19, R20, R9, RT1: footprint (none) -> Resistors:RESC1608N
- SW1: footprint (none) -> Switches:SW_CK-JS202011SCQN
- U5: footprint (none) -> SOT:SOT95P275-5L40N
- U6: footprint (none) -> QFN:QFN50P400X400-21T280X280N
