File: Hardware/Microcontroller.sch (KiCad schematic (older format))
At the start: 24 parts, among them J1 Conn_Cortex-JTAG-10, J2 Conn_USB-Mini, U2 STM32L151CBT, X1 8MHz, X2 32.768kHz

Commit message: Small changes
Parts:
- C10: footprint (none) -> Capacitors:CAPC2012N; Manufacturer Value -> Samsung; Manufacturer Part # Value -> CL21A106KPFNNNE; Vendor Value -> Digikey; Vendor Part # Value -> 1276-1052-1-ND
- C11, C12, C13, C14, C15, C16, C5, C6, C7, C8, C9: footprint (none) -> Capacitors:CAPC1608N
- D1, D2: footprint (none) -> LEDs:LEDC2012N
- FB1: footprint (none) -> Inductors:INDC1608N
- J1: footprint (none) -> Connectors:Conn_Samtec-FTSH-105-D-K
- J2: footprint (none) -> Connectors:Conn_USB-Mini-690-005-299-043
- PTC1: footprint (none) -> Resistors:RESC2012N
- R3, R4, R5: footprint (none) -> Resistors:RESC1608N
- U2: footprint (none) -> QFP:QFP50P900X900-48N
- X1: footprint (none) -> Clocks:Crystal_Abracon-ABM3
- X2: footprint (none) -> Clocks:Crystal_Abracon-ABS07

Commit message: Pinmapping
Parts:
- removed C11, C14: 18pF, Capacitors:CAPC1608N, symbol Capacitor
- removed X2: 32.768kHz, Clocks:Crystal_Abracon-ABS07, symbol Crystal
Connections:
- net GPS_RX: now also U2.21 (PB10)
- net GPS_TX: now also U2.22 (PB11)
- net XCVR_SCLK: now also U2.39 (PB3)
- net XCVR_SDI: now also U2.41 (PB5)
- net XCVR_SDO: now also U2.40 (PB4)
- net ~XCVR_CS: now also U2.38 (PA15)
- net VCO_EN: now reaches U2.13 (PA3)
Changed lines of the file:
@@
-$EndComp
-$Comp
-L Crystal X2
-U 1 1 5497A3B5
-P 3450 4800
-F 0 "X2" H 3450 4950 60  0000 C CNN
-F 1 "32.768kHz" H 3450 4650 60  0000 C CNN
-F 2 "Clocks:Crystal_Abracon-ABS07" H 3450 4800 60  0001 C CNN
-F 3 "" H 3450 4800 60  0000 C CNN
-F 4 "Abracon" H 3450 4800 60  0001 C CNN "Manufacturer"
-F 5 "ABS07-32.768KHZ-T" H 3450 4800 60  0001 C CNN "Manufacturer Part #"
-F 6 "Digikey" H 3450 4800 60  0001 C CNN "Vendor"
-F 7 "535-9542-1-ND" H 3450 4800 60  0001 C CNN "Vendor Part #"
-	1    3450 4800
-	1    0    0    -1
 $EndComp
 $Comp
@@
 Text Label 2000 4800 0    60   ~ 0
 OSC_O
-Text Label 3000 4800 2    60   ~ 0
-SOSC_I
-Text Label 3900 4800 0    60   ~ 0
-SOSC_O
-Wire Wire Line
-	3700 4800 3900 4800
-Wire Wire Line
-	3800 4900 3800 4800
-Connection ~ 3800 4800
-Wire Wire Line
-	3000 4800 3200 4800
-Wire Wire Line
-	3100 4900 3100 4800
-Connection ~ 3100 4800
 $Comp
 L GND #PWR07
-U 1 1 5497A6B2
-P 3450 5600
-F 0 "#PWR07" H 3450 5350 60  0001 C CNN
-F 1 "GND" H 3450 5450 60  0000 C CNN
-F 2 "" H 3450 5600 60  0000 C CNN
-F 3 "" H 3450 5600 60  0000 C CNN
-	1    3450 5600
-	1    0    0    -1
-$EndComp
-Wire Wire Line
-	3100 5400 3100 5500
-Wire Wire Line
-	3100 5500 3800 5500
-Wire Wire Line
-	3450 5500 3450 5600
-Wire Wire Line
-	3800 5500 3800 5400
-Connection ~ 3450 5500
-$Comp
-L GND #PWR08
 U 1 1 5497A76F
 P 1550 5600
-F 0 "#PWR08" H 1550 5350 60  0001 C CNN
+F 0 "#PWR07" H 1550 5350 60  0001 C CNN
 F 1 "GND" H 1550 5450 60  0000 C CNN
 F 2 "" H 1550 5600 60  0000 C CNN
@@
 VDDA
 Connection ~ 3700 6600
-Text HLabel 8500 5100 0    60   Output ~ 0
+Text HLabel 9100 4100 2    60   Output ~ 0
 GPS_RX
-Text HLabel 8500 5200 0    60   Input ~ 0
+Text HLabel 9100 4200 2    60   Input ~ 0
 GPS_TX
 Text HLabel 8500 5000 0    60   Output ~ 0
@@
 Connection ~ 3200 6600
 $Comp
-L GND #PWR09
+L GND #PWR08
 U 1 1 5497E456
 P 4400 7300
-F 0 "#PWR09" H 4400 7050 60  0001 C CNN
+F 0 "#PWR08" H 4400 7050 60  0001 C CNN
 F 1 "GND" H 4400 7150 60  0000 C CNN
 F 2 "" H 4400 7300 60  0000 C CNN
@@
 	4400 7300 4400 7200
 $Comp
-L GND #PWR010
+L GND #PWR09
 U 1 1 5497E541
 P 5000 7300
-F 0 "#PWR010" H 5000 7050 60  0001 C CNN
+F 0 "#PWR09" H 5000 7050 60  0001 C CNN
 F 1 "GND" H 5000 7150 60  0000 C CNN
 F 2 "" H 5000 7300 60  0000 C CNN
@@
 	1500 1900 1600 1900
 $Comp
-L GND #PWR011
+L GND #PWR010
 U 1 1 5497EA2C
 P 1600 2500
-F 0 "#PWR011" H 1600 2250 60  0001 C CNN
+F 0 "#PWR010" H 1600 2250 60  0001 C CNN
 F 1 "GND" H 1600 2350 60  0000 C CNN
 F 2 "" H 1600 2500 60  0000 C CNN
@@
 Connection ~ 1600 2100
 $Comp
-L GND #PWR012
+L GND #PWR011
 U 1 1 5497EF4B
 P 1000 7300
-F 0 "#PWR012" H 1000 7050 60  0001 C CNN
+F 0 "#PWR011" H 1000 7050 60  0001 C CNN
 F 1 "GND" H 1000 7150 60  0000 C CNN
 F 2 "" H 1000 7300 60  0000 C CNN
@@
 $EndComp
 $Comp
-L GND #PWR013
+L GND #PWR012
 U 1 1 5497EF5F
 P 1500 7300
-F 0 "#PWR013" H 1500 7050 60  0001 C CNN
+F 0 "#PWR012" H 1500 7050 60  0001 C CNN
 F 1 "GND" H 1500 7150 60  0000 C CNN
 F 2 "" H 1500 7300 60  0000 C CNN
@@
 $EndComp
 $Comp
-L GND #PWR014
+L GND #PWR013
 U 1 1 5497EF73
 P 2000 7300
-F 0 "#PWR014" H 2000 7050 60  0001 C CNN
+F 0 "#PWR013" H 2000 7050 60  0001 C CNN
 F 1 "GND" H 2000 7150 60  0000 C CNN
 F 2 "" H 2000 7300 60  0000 C CNN
@@
 $EndComp
 $Comp
-L GND #PWR015
+L GND #PWR014
 U 1 1 5497EF87
 P 2500 7300
-F 0 "#PWR015" H 2500 7050 60  0001 C CNN
+F 0 "#PWR014" H 2500 7050 60  0001 C CNN
 F 1 "GND" H 2500 7150 60  0000 C CNN
 F 2 "" H 2500 7300 60  0000 C CNN
@@
 $EndComp
 $Comp
-L GND #PWR016
+L GND #PWR015
 U 1 1 5497EF9B
 P 3200 7300
-F 0 "#PWR016" H 3200 7050 60  0001 C CNN
+F 0 "#PWR015" H 3200 7050 60  0001 C CNN
 F 1 "GND" H 3200 7150 60  0000 C CNN
 F 2 "" H 3200 7300 60  0000 C CNN
@@
 $EndComp
 $Comp
-L GND #PWR017
+L GND #PWR016
 U 1 1 5497EFAF
 P 3700 7300
-F 0 "#PWR017" H 3700 7050 60  0001 C CNN
+F 0 "#PWR016" H 3700 7050 60  0001 C CNN
 F 1 "GND" H 3700 7150 60  0000 C CNN
 F 2 "" H 3700 7300 60  0000 C CNN
@@
 ~RST
 $Comp
-L GND #PWR018
+L GND #PWR017
 U 1 1 549801E1
 P 1800 4100
-F 0 "#PWR018" H 1800 3850 60  0001 C CNN
+F 0 "#PWR017" H 1800 3850 60  0001 C CNN
 F 1 "GND" H 1800 3950 60  0000 C CNN
 F 2 "" H 1800 4100 60  0000 C CNN
@@
 Connection ~ 1800 4000
 $Comp
-L +3V3 #PWR019
+L +3V3 #PWR018
 U 1 1 5498032A
 P 1800 3100
-F 0 "#PWR019" H 1800 2950 60  0001 C CNN
+F 0 "#PWR018" H 1800 2950 60  0001 C CNN
 F 1 "+3V3" H 1800 3240 60  0000 C CNN
 F 2 "" H 1800 3100 60  0000 C CNN
@@
 	1800 3700 1700 3700
 $Comp
-L GND #PWR020
+L GND #PWR019
 U 1 1 54980CDC
 P 5600 7300
-F 0 "#PWR020" H 5600 7050 60  0001 C CNN
+F 0 "#PWR019" H 5600 7050 60  0001 C CNN
 F 1 "GND" H 5600 7150 60  0000 C CNN
 F 2 "" H 5600 7300 60  0000 C CNN
@@
 	4400 1200 4500 1200
 $Comp
-L +5VP #PWR021
+L +5VP #PWR020
 U 1 1 549925F2
 P 5100 1100
-F 0 "#PWR021" H 5100 950 60  0001 C CNN
+F 0 "#PWR020" H 5100 950 60  0001 C CNN
 F 1 "+5VP" H 5100 1240 60  0000 C CNN
 F 2 "" H 5100 1100 60  0000 C CNN
@@
 	5100 1200 5000 1200
 $Comp
-L GND #PWR022
+L GND #PWR021
 U 1 1 54992C8C
 P 4400 2000
-F 0 "#PWR022" H 4400 1750 60  0001 C CNN
+F 0 "#PWR021" H 4400 1750 60  0001 C CNN
 F 1 "GND" H 4400 1850 60  0000 C CNN
 F 2 "" H 4400 2000 60  0000 C CNN
@@
 Text HLabel 9500 5000 0    60   Output ~ 0
 XCVR_EN
-Text HLabel 9500 5100 0    60   Output ~ 0
+Text HLabel 9100 3400 2    60   Output ~ 0
 XCVR_SCLK
-Text HLabel 9500 5200 0    60   Output ~ 0
+Text HLabel 9100 3600 2    60   Output ~ 0
 XCVR_SDI
-Text HLabel 9500 5300 0    60   Input ~ 0
+Text HLabel 9100 3500 2    60   Input ~ 0
 XCVR_SDO
-Text HLabel 9500 5400 0    60   Output ~ 0
+Text HLabel 9100 2500 2    60   Output ~ 0
 ~XCVR_CS
-Text HLabel 9500 5500 0    60   Input ~ 0
+Text HLabel 9500 5100 0    60   Input ~ 0
 ~XCVR_INT
 Text HLabel 8500 6000 0    60   Input ~ 0
@@
 $EndComp
 $Comp
-L +3V3 #PWR023
+L +3V3 #PWR022
 U 1 1 54A1A643
 P 4200 3200
-F 0 "#PWR023" H 4200 3050 60  0001 C CNN
+F 0 "#PWR022" H 4200 3050 60  0001 C CNN
 F 1 "+3V3" H 4200 3340 60  0000 C CNN
 F 2 "" H 4200 3200 60  0000 C CNN
@@
 	1    5000 6950
 	0    1    1    0
-$EndComp
-$Comp
-L Capacitor C14
-U 1 1 54A2B687
-P 3800 5150
-F 0 "C14" V 3650 5250 60  0000 L CNN
-F 1 "18pF" V 3750 5250 60  0000 L CNN
-F 2 "Capacitors:CAPC1608N" H 3700 5150 60  0001 C CNN
-F 3 "" H 3800 5250 60  0001 C CNN
-F 4 "Samsung" H 3800 5150 60  0001 C CNN "Manufacturer"
-F 5 "CL10C180JB8NNNC" H 3800 5150 60  0001 C CNN "Manufacturer Part #"
-F 6 "Digikey" H 3800 5150 60  0001 C CNN "Vendor"
-F 7 "1276-1089-1-ND" H 3800 5150 60  0001 C CNN "Vendor Part #"
-F 8 "50V" V 3850 5250 50  0000 L CNN "Voltage"
-F 9 "NP0" V 3950 5250 50  0000 L CNN "Dielectric"
-	1    3800 5150
-	0    1    1    0
-$EndComp
-$Comp
-L Capacitor C11
-U 1 1 54A2B711
-P 3100 5150
-F 0 "C11" V 2950 5250 60  0000 L CNN
-F 1 "18pF" V 3050 5250 60  0000 L CNN
-F 2 "Capacitors:CAPC1608N" H 3000 5150 60  0001 C CNN
-F 3 "" H 3100 5250 60  0001 C CNN
-F 4 "Samsung" H 3100 5150 60  0001 C CNN "Manufacturer"
-F 5 "CL10C180JB8NNNC" H 3100 5150 60  0001 C CNN "Manufacturer Part #"
-F 6 "Digikey" H 3100 5150 60  0001 C CNN "Vendor"
-F 7 "1276-1089-1-ND" H 3100 5150 60  0001 C CNN "Vendor Part #"
-F 8 "50V" V 3150 5250 50  0000 L CNN "Voltage"
-F 9 "NP0" V 3250 5250 50  0000 L CNN "Dielectric"
-	1    3100 5150
-	0    -1   1    0
 $EndComp
 $Comp
@@
 	0    1    1    0
 $EndComp
+Wire Wire Line
+	9000 4100 9100 4100
+Wire Wire Line
+	9100 4200 9000 4200
+Text HLabel 9400 1300 2    60   Output ~ 0
+VCO_EN
+Wire Wire Line
+	9400 1300 9000 1300
+Wire Wire Line
+	9100 2500 9000 2500
+Wire Wire Line
+	9100 3400 9000 3400
+Wire Wire Line
+	9000 3500 9100 3500
+Wire Wire Line
+	9100 3600 9000 3600
 $EndSCHEMATC
