File: Hardware/Radio.sch (KiCad schematic (older format))
At the start: 25 parts, among them J3 Conn_Coax, U3 Si4464, U4 AS213, X3 27MHz

Commit message: BOM fields
Parts:
- C20, C22, C26: Dielectric X5R -> X7R; Manufacturer Value -> Samsung; Manufacturer Part # Value -> CL10B104KO8NNNC; Vendor Value -> Digikey; Vendor Part # Value -> 1276-1005-1-ND; Voltage 10V -> 16V
- C21: value 2.2uF -> 1uF; Dielectric X5R -> X7R; Manufacturer Value -> Samsung; Manufacturer Part # Value -> CL10B105KP8NNNC; Vendor Value -> Digikey; Vendor Part # Value -> 1276-1946-1-ND
- R7, R8: value 10k -> 100k; Manufacturer Value -> Yageo; Manufacturer Part # Value -> RC0603JR-07100KL; Vendor Value -> Digikey; Vendor Part # Value -> 311-100KGRCT-ND
- U3: Manufacturer (none) -> Silicon Labratories; Manufacturer Part # (none) -> SI4464-B1B-FM; Vendor (none) -> Digikey; Vendor Part # (none) -> 336-2472-5-ND
Changed lines of the file:
@@
 F 2 "" H 2250 1550 60  0000 C CNN
 F 3 "" H 2250 1550 60  0000 C CNN
+F 4 "Silicon Labratories" H 2250 1550 60  0001 C CNN "Manufacturer"
+F 5 "SI4464-B1B-FM" H 2250 1550 60  0001 C CNN "Manufacturer Part #"
+F 6 "Digikey" H 2250 1550 60  0001 C CNN "Vendor"
+F 7 "336-2472-5-ND" H 2250 1550 60  0001 C CNN "Vendor Part #"
 	1    2250 1550
 	1    0    0    -1
-$EndComp
-$Comp
-L Capacitor C21
-U 1 1 5498E23C
-P 4600 1550
-F 0 "C21" V 4450 1650 60  0000 L CNN
-F 1 "2.2uF" V 4550 1650 60  0000 L CNN
-F 2 "" H 4500 1550 60  0001 C CNN
-F 3 "" H 4600 1650 60  0001 C CNN
-F 4 "Value" H 4600 1550 60  0001 C CNN "Manufacturer"
-F 5 "Value" H 4600 1550 60  0001 C CNN "Manufacturer Part #"
-F 6 "Value" H 4600 1550 60  0001 C CNN "Vendor"
-F 7 "Value" H 4600 1550 60  0001 C CNN "Vendor Part #"
-F 8 "10V" V 4650 1650 50  0000 L CNN "Voltage"
-F 9 "X5R" V 4750 1650 50  0000 L CNN "Dielectric"
-	1    4600 1550
-	0    -1   1    0
-$EndComp
-$Comp
-L Capacitor C20
-U 1 1 5498E2A6
-P 4100 1550
-F 0 "C20" V 3950 1650 60  0000 L CNN
-F 1 "0.1uF" V 4050 1650 60  0000 L CNN
-F 2 "" H 4000 1550 60  0001 C CNN
-F 3 "" H 4100 1650 60  0001 C CNN
-F 4 "Value" H 4100 1550 60  0001 C CNN "Manufacturer"
-F 5 "Value" H 4100 1550 60  0001 C CNN "Manufacturer Part #"
-F 6 "Value" H 4100 1550 60  0001 C CNN "Vendor"
-F 7 "Value" H 4100 1550 60  0001 C CNN "Vendor Part #"
-F 8 "10V" V 4150 1650 50  0000 L CNN "Voltage"
-F 9 "X5R" V 4250 1650 50  0000 L CNN "Dielectric"
-	1    4100 1550
-	0    -1   1    0
 $EndComp
 $Comp
@@
 	1    0    0    1
 $EndComp
-$Comp
-L Capacitor C22
-U 1 1 5498E392
-P 5300 1550
-F 0 "C22" V 5150 1650 60  0000 L CNN
-F 1 "0.1uF" V 5250 1650 60  0000 L CNN
-F 2 "" H 5200 1550 60  0001 C CNN
-F 3 "" H 5300 1650 60  0001 C CNN
-F 4 "Value" H 5300 1550 60  0001 C CNN "Manufacturer"
-F 5 "Value" H 5300 1550 60  0001 C CNN "Manufacturer Part #"
-F 6 "Value" H 5300 1550 60  0001 C CNN "Vendor"
-F 7 "Value" H 5300 1550 60  0001 C CNN "Vendor Part #"
-F 8 "10V" V 5350 1650 50  0000 L CNN "Voltage"
-F 9 "X5R" V 5450 1650 50  0000 L CNN "Dielectric"
-	1    5300 1550
-	0    1    1    0
-$EndComp
 Text Label 5300 1100 1    60   ~ 0
 VDDA
@@
 $EndComp
 $Comp
-L Capacitor C26
-U 1 1 549DC500
-P 8700 1750
-F 0 "C26" V 8550 1850 60  0000 L CNN
-F 1 "0.1uF" V 8650 1850 60  0000 L CNN
-F 2 "" H 8600 1750 60  0001 C CNN
-F 3 "" H 8700 1850 60  0001 C CNN
-F 4 "Value" H 8700 1750 60  0001 C CNN "Manufacturer"
-F 5 "Value" H 8700 1750 60  0001 C CNN "Manufacturer Part #"
-F 6 "Value" H 8700 1750 60  0001 C CNN "Vendor"
-F 7 "Value" H 8700 1750 60  0001 C CNN "Vendor Part #"
-F 8 "10V" V 8750 1850 50  0000 L CNN "Voltage"
-F 9 "X5R" V 8850 1850 50  0000 L CNN "Dielectric"
-	1    8700 1750
-	0    1    1    0
-$EndComp
-$Comp
 L GND #PWR34
 U 1 1 549DC55A
@@
 	8700 1300 8700 1500
 Connection ~ 8500 1300
-$Comp
-L Resistor R7
-U 1 1 549DC7C7
-P 9050 1200
-F 0 "R7" V 8900 1300 60  0000 L CNN
-F 1 "10k" V 9000 1300 60  0000 L CNN
-F 2 "" H 8950 1200 60  0001 C CNN
-F 3 "" H 9050 1300 60  0001 C CNN
-F 4 "Value" H 9050 1200 60  0001 C CNN "Manufacturer"
-F 5 "Value" H 9050 1200 60  0001 C CNN "Manufacturer Part #"
-F 6 "Value" H 9050 1200 60  0001 C CNN "Vendor"
-F 7 "Value" H 9050 1200 60  0001 C CNN "Vendor Part #"
-F 8 "1/10W" V 9100 1300 50  0000 L CNN "Power"
-F 9 "5%" V 9200 1300 50  0000 L CNN "Tolerance"
-	1    9050 1200
-	1    0    0    -1
-$EndComp
-$Comp
-L Resistor R8
-U 1 1 549DC844
-P 9400 1550
-F 0 "R8" V 9250 1650 60  0000 L CNN
-F 1 "10k" V 9350 1650 60  0000 L CNN
-F 2 "" H 9300 1550 60  0001 C CNN
-F 3 "" H 9400 1650 60  0001 C CNN
-F 4 "Value" H 9400 1550 60  0001 C CNN "Manufacturer"
-F 5 "Value" H 9400 1550 60  0001 C CNN "Manufacturer Part #"
-F 6 "Value" H 9400 1550 60  0001 C CNN "Vendor"
-F 7 "Value" H 9400 1550 60  0001 C CNN "Vendor Part #"
-F 8 "1/10W" V 9450 1650 50  0000 L CNN "Power"
-F 9 "5%" V 9550 1650 50  0000 L CNN "Tolerance"
-	1    9400 1550
-	0    1    1    0
-$EndComp
 $Comp
 L Capacitor C28
@@
 Wire Wire Line
 	6100 3900 6000 3900
+$Comp
+L Resistor R8
+U 1 1 54A25AF9
+P 9400 1550
+F 0 "R8" V 9250 1650 60  0000 L CNN
+F 1 "100k" V 9350 1650 60  0000 L CNN
+F 2 "" H 9300 1550 60  0001 C CNN
+F 3 "" H 9400 1650 60  0001 C CNN
+F 4 "Yageo" H 9400 1550 60  0001 C CNN "Manufacturer"
+F 5 "RC0603JR-07100KL" H 9400 1550 60  0001 C CNN "Manufacturer Part #"
+F 6 "Digikey" H 9400 1550 60  0001 C CNN "Vendor"
+F 7 "311-100KGRCT-ND" H 9400 1550 60  0001 C CNN "Vendor Part #"
+F 8 "1/10W" V 9450 1650 50  0000 L CNN "Power"
+F 9 "5%" V 9550 1650 50  0000 L CNN "Tolerance"
+	1    9400 1550
+	0    1    1    0
+$EndComp
+$Comp
+L Resistor R7
+U 1 1 54A25CB1
+P 9050 1200
+F 0 "R7" V 8900 1300 60  0000 L CNN
+F 1 "100k" V 9000 1300 60  0000 L CNN
+F 2 "" H 8950 1200 60  0001 C CNN
+F 3 "" H 9050 1300 60  0001 C CNN
+F 4 "Yageo" H 9050 1200 60  0001 C CNN "Manufacturer"
+F 5 "RC0603JR-07100KL" H 9050 1200 60  0001 C CNN "Manufacturer Part #"
+F 6 "Digikey" H 9050 1200 60  0001 C CNN "Vendor"
+F 7 "311-100KGRCT-ND" H 9050 1200 60  0001 C CNN "Vendor Part #"
+F 8 "1/10W" V 9100 1300 50  0000 L CNN "Power"
+F 9 "5%" V 9200 1300 50  0000 L CNN "Tolerance"
+	1    9050 1200
+	1    0    0    -1
+$EndComp
+$Comp
+L Capacitor C22
+U 1 1 54A29C62
+P 5300 1550
+F 0 "C22" V 5150 1650 60  0000 L CNN
+F 1 "0.1uF" V 5250 1650 60  0000 L CNN
+F 2 "" H 5200 1550 60  0001 C CNN
+F 3 "" H 5300 1650 60  0001 C CNN
+F 4 "Samsung" H 5300 1550 60  0001 C CNN "Manufacturer"
+F 5 "CL10B104KO8NNNC" H 5300 1550 60  0001 C CNN "Manufacturer Part #"
+F 6 "Digikey" H 5300 1550 60  0001 C CNN "Vendor"
+F 7 "1276-1005-1-ND" H 5300 1550 60  0001 C CNN "Vendor Part #"
+F 8 "16V" V 5350 1650 50  0000 L CNN "Voltage"
+F 9 "X7R" V 5450 1650 50  0000 L CNN "Dielectric"
+	1    5300 1550
+	0    1    1    0
+$EndComp
+$Comp
+L Capacitor C20
+U 1 1 54A29CEB
+P 4100 1550
+F 0 "C20" V 3950 1650 60  0000 L CNN
+F 1 "0.1uF" V 4050 1650 60  0000 L CNN
+F 2 "" H 4000 1550 60  0001 C CNN
+F 3 "" H 4100 1650 60  0001 C CNN
+F 4 "Samsung" H 4100 1550 60  0001 C CNN "Manufacturer"
+F 5 "CL10B104KO8NNNC" H 4100 1550 60  0001 C CNN "Manufacturer Part #"
+F 6 "Digikey" H 4100 1550 60  0001 C CNN "Vendor"
+F 7 "1276-1005-1-ND" H 4100 1550 60  0001 C CNN "Vendor Part #"
+F 8 "16V" V 4150 1650 50  0000 L CNN "Voltage"
+F 9 "X7R" V 4250 1650 50  0000 L CNN "Dielectric"
+	1    4100 1550
+	0    -1   1    0
+$EndComp
+$Comp
+L Capacitor C26
+U 1 1 54A29D58
+P 8700 1750
+F 0 "C26" V 8550 1850 60  0000 L CNN
+F 1 "0.1uF" V 8650 1850 60  0000 L CNN
+F 2 "" H 8600 1750 60  0001 C CNN
+F 3 "" H 8700 1850 60  0001 C CNN
+F 4 "Samsung" H 8700 1750 60  0001 C CNN "Manufacturer"
+F 5 "CL10B104KO8NNNC" H 8700 1750 60  0001 C CNN "Manufacturer Part #"
+F 6 "Digikey" H 8700 1750 60  0001 C CNN "Vendor"
+F 7 "1276-1005-1-ND" H 8700 1750 60  0001 C CNN "Vendor Part #"
+F 8 "16V" V 8750 1850 50  0000 L CNN "Voltage"
+F 9 "X7R" V 8850 1850 50  0000 L CNN "Dielectric"
+	1    8700 1750
+	0    1    1    0
+$EndComp
+$Comp
+L Capacitor C21
+U 1 1 54A2A9C3
+P 4600 1550
+F 0 "C21" V 4450 1650 60  0000 L CNN
+F 1 "1uF" V 4550 1650 60  0000 L CNN
+F 2 "" H 4500 1550 60  0001 C CNN
+F 3 "" H 4600 1650 60  0001 C CNN
+F 4 "Samsung" H 4600 1550 60  0001 C CNN "Manufacturer"
+F 5 "CL10B105KP8NNNC" H 4600 1550 60  0001 C CNN "Manufacturer Part #"
+F 6 "Digikey" H 4600 1550 60  0001 C CNN "Vendor"
+F 7 "1276-1946-1-ND" H 4600 1550 60  0001 C CNN "Vendor Part #"
+F 8 "10V" V 4650 1650 50  0000 L CNN "Voltage"
+F 9 "X7R" V 4750 1650 50  0000 L CNN "Dielectric"
+	1    4600 1550
+	0    -1   1    0
+$EndComp
 $EndSCHEMATC

Commit message: Small changes
Parts:
- C17, C18, C19, C20, C21, C22, C23, C24, C25, C26, C27, C28: footprint (none) -> Capacitors:CAPC1608N
- FB2, L2, L3, L4, L5, L6: footprint (none) -> Inductors:INDC1608N
- J3: footprint (none) -> Connectors:Conn_RF_Linx-CONSMA003.031-L
- R6, R7, R8: footprint (none) -> Resistors:RESC1608N
- U3: footprint (none) -> QFN:QFN50P400X400-21T275X275N
- U4: footprint (none) -> SOT:SOT65P220-6N
- X3: footprint (none) -> Clocks:Osc_CTS-357
Changed lines of the file:
@@
 F 0 "U3" H 2250 2200 60  0000 C CNN
 F 1 "Si4464" H 2250 900 60  0000 C CNN
-F 2 "" H 2250 1550 60  0000 C CNN
+F 2 "QFN:QFN50P400X400-21T275X275N" H 2250 1550 60  0001 C CNN
 F 3 "" H 2250 1550 60  0000 C CNN
 F 4 "Silicon Labratories" H 2250 1550 60  0001 C CNN "Manufacturer"
@@
 F 0 "FB2" V 4800 1300 60  0000 L CNN
 F 1 "Ferrite" V 4900 1300 60  0000 L CNN
-F 2 "" H 4850 1200 60  0001 C CNN
+F 2 "Inductors:INDC1608N" H 4850 1200 60  0001 C CNN
 F 3 "" H 4950 1300 60  0001 C CNN
 F 4 "Value" H 4950 1200 60  0001 C CNN "Manufacturer"
@@
 VDD
 $Comp
-L +3V3 #PWR27
+L +3V3 #PWR024
 U 1 1 5498E41D
 P 4600 1100
-F 0 "#PWR27" H 4600 950 60  0001 C CNN
+F 0 "#PWR024" H 4600 950 60  0001 C CNN
 F 1 "+3V3" H 4600 1240 60  0000 C CNN
 F 2 "" H 4600 1100 60  0000 C CNN
@@
 Connection ~ 4100 1200
 $Comp
-L GND #PWR26
+L GND #PWR025
 U 1 1 5498E46B
 P 4100 1900
-F 0 "#PWR26" H 4100 1650 60  0001 C CNN
+F 0 "#PWR025" H 4100 1650 60  0001 C CNN
 F 1 "GND" H 4100 1750 60  0000 C CNN
 F 2 "" H 4100 1900 60  0000 C CNN
@@
 $EndComp
 $Comp
-L GND #PWR28
+L GND #PWR026
 U 1 1 5498E47F
 P 4600 1900
-F 0 "#PWR28" H 4600 1650 60  0001 C CNN
+F 0 "#PWR026" H 4600 1650 60  0001 C CNN
 F 1 "GND" H 4600 1750 60  0000 C CNN
 F 2 "" H 4600 1900 60  0000 C CNN
@@
 $EndComp
 $Comp
-L GND #PWR29
+L GND #PWR027
 U 1 1 5498E493
 P 5300 1900
-F 0 "#PWR29" H 5300 1650 60  0001 C CNN
+F 0 "#PWR027" H 5300 1650 60  0001 C CNN
 F 1 "GND" H 5300 1750 60  0000 C CNN
 F 2 "" H 5300 1900 60  0000 C CNN
@@
 VDDA
 $Comp
-L GND #PWR25
+L GND #PWR028
 U 1 1 5498E5DD
 P 2900 2200
-F 0 "#PWR25" H 2900 1950 60  0001 C CNN
+F 0 "#PWR028" H 2900 1950 60  0001 C CNN
 F 1 "GND" H 2900 2050 60  0000 C CNN
 F 2 "" H 2900 2200 60  0000 C CNN
@@
 F 0 "L2" V 1350 3450 60  0000 L CNN
 F 1 "Inductor" V 1450 3450 60  0000 L CNN
-F 2 "" H 1400 3350 60  0001 C CNN
+F 2 "Inductors:INDC1608N" H 1400 3350 60  0001 C CNN
 F 3 "" H 1500 3450 60  0001 C CNN
 F 4 "Value" H 1500 3350 60  0001 C CNN "Manufacturer"
@@
 F 0 "L3" V 1700 3800 60  0000 L CNN
 F 1 "Inductor" V 1800 3800 60  0000 L CNN
-F 2 "" H 1750 3700 60  0001 C CNN
+F 2 "Inductors:INDC1608N" H 1750 3700 60  0001 C CNN
 F 3 "" H 1850 3800 60  0001 C CNN
 F 4 "Value" H 1850 3700 60  0001 C CNN "Manufacturer"
@@
 F 0 "C17" V 1350 4150 60  0000 L CNN
 F 1 "Capacitor" V 1450 4150 60  0000 L CNN
-F 2 "" H 1400 4050 60  0001 C CNN
+F 2 "Capacitors:CAPC1608N" H 1400 4050 60  0001 C CNN
 F 3 "" H 1500 4150 60  0001 C CNN
 F 4 "Value" H 1500 4050 60  0001 C CNN "Manufacturer"
@@
 F 0 "C18" V 1700 3100 60  0000 L CNN
 F 1 "Capacitor" V 1800 3100 60  0000 L CNN
-F 2 "" H 1750 3000 60  0001 C CNN
+F 2 "Capacitors:CAPC1608N" H 1750 3000 60  0001 C CNN
 F 3 "" H 1850 3100 60  0001 C CNN
 F 4 "Value" H 1850 3000 60  0001 C CNN "Manufacturer"
@@
 RXn
 $Comp
-L GND #PWR24
+L GND #PWR029
 U 1 1 5498F76A
 P 1500 4400
-F 0 "#PWR24" H 1500 4150 60  0001 C CNN
+F 0 "#PWR029" H 1500 4150 60  0001 C CNN
 F 1 "GND" H 1500 4250 60  0000 C CNN
 F 2 "" H 1500 4400 60  0000 C CNN
@@
 F 0 "X3" H 7900 1500 60  0000 C CNN
 F 1 "27MHz" H 7900 1100 60  0000 C CNN
-F 2 "" H 7900 1300 60  0000 C CNN
+F 2 "Clocks:Osc_CTS-357" H 7900 1300 60  0001 C CNN
 F 3 "" H 7900 1300 60  0000 C CNN
 F 4 "CTS" H 7900 1300 60  0001 C CNN "Manufacturer"
@@
 $EndComp
 $Comp
-L GND #PWR34
+L GND #PWR030
 U 1 1 549DC55A
 P 8500 2200
-F 0 "#PWR34" H 8500 1950 60  0001 C CNN
+F 0 "#PWR030" H 8500 1950 60  0001 C CNN
 F 1 "GND" H 8500 2050 60  0000 C CNN
 F 2 "" H 8500 2200 60  0000 C CNN
@@
 Connection ~ 8500 2100
 $Comp
-L +3V3 #PWR33
+L +3V3 #PWR031
 U 1 1 549DC644
 P 8500 1100
-F 0 "#PWR33" H 8500 950 60  0001 C CNN
+F 0 "#PWR031" H 8500 950 60  0001 C CNN
 F 1 "+3V3" H 8500 1240 60  0000 C CNN
 F 2 "" H 8500 1100 60  0000 C CNN
@@
 F 0 "C28" V 9600 1300 60  0000 L CNN
 F 1 "0.01uF" V 9700 1300 60  0000 L CNN
-F 2 "" H 9650 1200 60  0001 C CNN
+F 2 "Capacitors:CAPC1608N" H 9650 1200 60  0001 C CNN
 F 3 "" H 9750 1300 60  0001 C CNN
 F 4 "Value" H 9750 1200 60  0001 C CNN "Manufacturer"
@@
 Connection ~ 9400 1200
 $Comp
-L GND #PWR36
+L GND #PWR032
 U 1 1 549DCA64
 P 9400 1900
-F 0 "#PWR36" H 9400 1650 60  0001 C CNN
+F 0 "#PWR032" H 9400 1650 60  0001 C CNN
 F 1 "GND" H 9400 1750 60  0000 C CNN
 F 2 "" H 9400 1900 60  0000 C CNN
@@
 F 0 "C24" V 7150 1850 60  0000 L CNN
 F 1 "0.01uF" V 7250 1850 60  0000 L CNN
-F 2 "" H 7200 1750 60  0001 C CNN
+F 2 "Capacitors:CAPC1608N" H 7200 1750 60  0001 C CNN
 F 3 "" H 7300 1850 60  0001 C CNN
 F 4 "Value" H 7300 1750 60  0001 C CNN "Manufacturer"
@@
 F 0 "R6" V 6800 1500 60  0000 L CNN
 F 1 "160" V 6900 1500 60  0000 L CNN
-F 2 "" H 6850 1400 60  0001 C CNN
+F 2 "Resistors:RESC1608N" H 6850 1400 60  0001 C CNN
 F 3 "" H 6950 1500 60  0001 C CNN
 F 4 "Value" H 6950 1400 60  0001 C CNN "Manufacturer"
@@
 Connection ~ 7300 1400
 $Comp
-L GND #PWR31
+L GND #PWR033
 U 1 1 549DD4D8
 P 7300 2100
-F 0 "#PWR31" H 7300 1850 60  0001 C CNN
+F 0 "#PWR033" H 7300 1850 60  0001 C CNN
 F 1 "GND" H 7300 1950 60  0000 C CNN
 F 2 "" H 7300 2100 60  0000 C CNN
@@
 F 0 "U4" H 6500 4000 60  0000 C CNN
 F 1 "AS213" H 6500 3500 60  0000 C CNN
-F 2 "" H 6500 3750 60  0000 C CNN
+F 2 "SOT:SOT65P220-6N" H 6500 3750 60  0001 C CNN
 F 3 "" H 6500 3750 60  0000 C CNN
 	1    6500 3750
@@
 RX
 $Comp
-L GND #PWR30
+L GND #PWR034
 U 1 1 549DFFDB
 P 7000 4000
-F 0 "#PWR30" H 7000 3750 60  0001 C CNN
+F 0 "#PWR034" H 7000 3750 60  0001 C CNN
 F 1 "GND" H 7000 3850 60  0000 C CNN
 F 2 "" H 7000 4000 60  0000 C CNN
@@
 F 0 "C19" V 2400 3800 60  0000 L CNN
 F 1 "470pF" V 2500 3800 60  0000 L CNN
-F 2 "" H 2450 3700 60  0001 C CNN
+F 2 "Capacitors:CAPC1608N" H 2450 3700 60  0001 C CNN
 F 3 "" H 2550 3800 60  0001 C CNN
 F 4 "Value" H 2550 3700 60  0001 C CNN "Manufacturer"
@@
 F 0 "C23" V 7100 3700 60  0000 L CNN
 F 1 "470pF" V 7200 3700 60  0000 L CNN
-F 2 "" H 7150 3600 60  0001 C CNN
+F 2 "Capacitors:CAPC1608N" H 7150 3600 60  0001 C CNN
 F 3 "" H 7250 3700 60  0001 C CNN
 F 4 "Value" H 7250 3600 60  0001 C CNN "Manufacturer"
@@
 F 0 "L4" V 7700 3700 60  0000 L CNN
 F 1 "Inductor" V 7800 3700 60  0000 L CNN
-F 2 "" H 7750 3600 60  0001 C CNN
+F 2 "Inductors:INDC1608N" H 7750 3600 60  0001 C CNN
 F 3 "" H 7850 3700 60  0001 C CNN
 F 4 "Value" H 7850 3600 60  0001 C CNN "Manufacturer"
@@
 F 0 "L5" V 8400 3700 60  0000 L CNN
 F 1 "Inductor" V 8500 3700 60  0000 L CNN
-F 2 "" H 8450 3600 60  0001 C CNN
+F 2 "Inductors:INDC1608N" H 8450 3600 60  0001 C CNN
 F 3 "" H 8550 3700 60  0001 C CNN
 F 4 "Value" H 8550 3600 60  0001 C CNN "Manufacturer"
@@
 F 0 "L6" V 9100 3700 60  0000 L CNN
 F 1 "Inductor" V 9200 3700 60  0000 L CNN
-F 2 "" H 9150 3600 60  0001 C CNN
+F 2 "Inductors:INDC1608N" H 9150 3600 60  0001 C CNN
 F 3 "" H 9250 3700 60  0001 C CNN
 F 4 "Value" H 9250 3600 60  0001 C CNN "Manufacturer"
@@
 F 0 "C25" V 8050 4050 60  0000 L CNN
 F 1 "Capacitor" V 8150 4050 60  0000 L CNN
-F 2 "" H 8100 3950 60  0001 C CNN
+F 2 "Capacitors:CAPC1608N" H 8100 3950 60  0001 C CNN
 F 3 "" H 8200 4050 60  0001 C CNN
 F 4 "Value" H 8200 3950 60  0001 C CNN "Manufacturer"
@@
 F 0 "C27" V 8750 4050 60  0000 L CNN
 F 1 "Capacitor" V 8850 4050 60  0000 L CNN
-F 2 "" H 8800 3950 60  0001 C CNN
+F 2 "Capacitors:CAPC1608N" H 8800 3950 60  0001 C CNN
 F 3 "" H 8900 4050 60  0001 C CNN
 F 4 "Value" H 8900 3950 60  0001 C CNN "Manufacturer"
@@
 F 0 "J3" H 9900 3850 60  0000 C CNN
 F 1 "Conn_Coax" H 9900 3750 60  0000 C CNN
-F 2 "" H 9900 3600 60  0000 C CNN
+F 2 "Connectors:Conn_RF_Linx-CONSMA003.031-L" H 9900 3600 60  0001 C CNN
 F 3 "" H 9900 3600 60  0000 C CNN
 	1    9900 3600
@@
 $EndComp
 $Comp
-L GND #PWR37
+L GND #PWR035
 U 1 1 549E0E20
 P 9600 3900
-F 0 "#PWR37" H 9600 3650 60  0001 C CNN
+F 0 "#PWR035" H 9600 3650 60  0001 C CNN
 F 1 "GND" H 9600 3750 60  0000 C CNN
 F 2 "" H 9600 3900 60  0000 C CNN
@@
 	9500 3600 9700 3600
 $Comp
-L GND #PWR35
+L GND #PWR036
 U 1 1 549E0F20
 P 8900 4300
-F 0 "#PWR35" H 8900 4050 60  0001 C CNN
+F 0 "#PWR036" H 8900 4050 60  0001 C CNN
 F 1 "GND" H 8900 4150 60  0000 C CNN
 F 2 "" H 8900 4300 60  0000 C CNN
@@
 $EndComp
 $Comp
-L GND #PWR32
+L GND #PWR037
 U 1 1 549E0F34
 P 8200 4300
-F 0 "#PWR32" H 8200 4050 60  0001 C CNN
+F 0 "#PWR037" H 8200 4050 60  0001 C CNN
 F 1 "GND" H 8200 4150 60  0000 C CNN
 F 2 "" H 8200 4300 60  0000 C CNN
@@
 F 0 "R8" V 9250 1650 60  0000 L CNN
 F 1 "100k" V 9350 1650 60  0000 L CNN
-F 2 "" H 9300 1550 60  0001 C CNN
+F 2 "Resistors:RESC1608N" H 9300 1550 60  0001 C CNN
 F 3 "" H 9400 1650 60  0001 C CNN
 F 4 "Yageo" H 9400 1550 60  0001 C CNN "Manufacturer"
@@
 F 0 "R7" V 8900 1300 60  0000 L CNN
 F 1 "100k" V 9000 1300 60  0000 L CNN
-F 2 "" H 8950 1200 60  0001 C CNN
+F 2 "Resistors:RESC1608N" H 8950 1200 60  0001 C CNN
 F 3 "" H 9050 1300 60  0001 C CNN
 F 4 "Yageo" H 9050 1200 60  0001 C CNN "Manufacturer"
@@
 F 0 "C22" V 5150 1650 60  0000 L CNN
 F 1 "0.1uF" V 5250 1650 60  0000 L CNN
-F 2 "" H 5200 1550 60  0001 C CNN
+F 2 "Capacitors:CAPC1608N" H 5200 1550 60  0001 C CNN
 F 3 "" H 5300 1650 60  0001 C CNN
 F 4 "Samsung" H 5300 1550 60  0001 C CNN "Manufacturer"
@@
 F 0 "C20" V 3950 1650 60  0000 L CNN
 F 1 "0.1uF" V 4050 1650 60  0000 L CNN
-F 2 "" H 4000 1550 60  0001 C CNN
+F 2 "Capacitors:CAPC1608N" H 4000 1550 60  0001 C CNN
 F 3 "" H 4100 1650 60  0001 C CNN
 F 4 "Samsung" H 4100 1550 60  0001 C CNN "Manufacturer"
@@
 F 0 "C26" V 8550 1850 60  0000 L CNN
 F 1 "0.1uF" V 8650 1850 60  0000 L CNN
-F 2 "" H 8600 1750 60  0001 C CNN
+F 2 "Capacitors:CAPC1608N" H 8600 1750 60  0001 C CNN
 F 3 "" H 8700 1850 60  0001 C CNN
 F 4 "Samsung" H 8700 1750 60  0001 C CNN "Manufacturer"
@@
 F 0 "C21" V 4450 1650 60  0000 L CNN
 F 1 "1uF" V 4550 1650 60  0000 L CNN
-F 2 "" H 4500 1550 60  0001 C CNN
+F 2 "Capacitors:CAPC1608N" H 4500 1550 60  0001 C CNN
 F 3 "" H 4600 1650 60  0001 C CNN
 F 4 "Samsung" H 4600 1550 60  0001 C CNN "Manufacturer"

Commit message: Pinmapping
Connections:
- net TxRamp: now reaches U3.7 (TXRAMP)
Changed lines of the file:
@@
 VDD
 $Comp
-L +3V3 #PWR024
+L +3V3 #PWR023
 U 1 1 5498E41D
 P 4600 1100
-F 0 "#PWR024" H 4600 950 60  0001 C CNN
+F 0 "#PWR023" H 4600 950 60  0001 C CNN
 F 1 "+3V3" H 4600 1240 60  0000 C CNN
 F 2 "" H 4600 1100 60  0000 C CNN
@@
 Connection ~ 4100 1200
 $Comp
-L GND #PWR025
+L GND #PWR024
 U 1 1 5498E46B
 P 4100 1900
-F 0 "#PWR025" H 4100 1650 60  0001 C CNN
+F 0 "#PWR024" H 4100 1650 60  0001 C CNN
 F 1 "GND" H 4100 1750 60  0000 C CNN
 F 2 "" H 4100 1900 60  0000 C CNN
@@
 $EndComp
 $Comp
-L GND #PWR026
+L GND #PWR025
 U 1 1 5498E47F
 P 4600 1900
-F 0 "#PWR026" H 4600 1650 60  0001 C CNN
+F 0 "#PWR025" H 4600 1650 60  0001 C CNN
 F 1 "GND" H 4600 1750 60  0000 C CNN
 F 2 "" H 4600 1900 60  0000 C CNN
@@
 $EndComp
 $Comp
-L GND #PWR027
+L GND #PWR026
 U 1 1 5498E493
 P 5300 1900
-F 0 "#PWR027" H 5300 1650 60  0001 C CNN
+F 0 "#PWR026" H 5300 1650 60  0001 C CNN
 F 1 "GND" H 5300 1750 60  0000 C CNN
 F 2 "" H 5300 1900 60  0000 C CNN
@@
 VDDA
 $Comp
-L GND #PWR028
+L GND #PWR027
 U 1 1 5498E5DD
 P 2900 2200
-F 0 "#PWR028" H 2900 1950 60  0001 C CNN
+F 0 "#PWR027" H 2900 1950 60  0001 C CNN
 F 1 "GND" H 2900 2050 60  0000 C CNN
 F 2 "" H 2900 2200 60  0000 C CNN
@@
 RXn
 $Comp
-L GND #PWR029
+L GND #PWR028
 U 1 1 5498F76A
 P 1500 4400
-F 0 "#PWR029" H 1500 4150 60  0001 C CNN
+F 0 "#PWR028" H 1500 4150 60  0001 C CNN
 F 1 "GND" H 1500 4250 60  0000 C CNN
 F 2 "" H 1500 4400 60  0000 C CNN
@@
 $EndComp
 $Comp
-L GND #PWR030
+L GND #PWR029
 U 1 1 549DC55A
 P 8500 2200
-F 0 "#PWR030" H 8500 1950 60  0001 C CNN
+F 0 "#PWR029" H 8500 1950 60  0001 C CNN
 F 1 "GND" H 8500 2050 60  0000 C CNN
 F 2 "" H 8500 2200 60  0000 C CNN
@@
 Connection ~ 8500 2100
 $Comp
-L +3V3 #PWR031
+L +3V3 #PWR030
 U 1 1 549DC644
 P 8500 1100
-F 0 "#PWR031" H 8500 950 60  0001 C CNN
+F 0 "#PWR030" H 8500 950 60  0001 C CNN
 F 1 "+3V3" H 8500 1240 60  0000 C CNN
 F 2 "" H 8500 1100 60  0000 C CNN
@@
 Connection ~ 9400 1200
 $Comp
-L GND #PWR032
+L GND #PWR031
 U 1 1 549DCA64
 P 9400 1900
-F 0 "#PWR032" H 9400 1650 60  0001 C CNN
+F 0 "#PWR031" H 9400 1650 60  0001 C CNN
 F 1 "GND" H 9400 1750 60  0000 C CNN
 F 2 "" H 9400 1900 60  0000 C CNN
@@
 Connection ~ 7300 1400
 $Comp
-L GND #PWR033
+L GND #PWR032
 U 1 1 549DD4D8
 P 7300 2100
-F 0 "#PWR033" H 7300 1850 60  0001 C CNN
+F 0 "#PWR032" H 7300 1850 60  0001 C CNN
 F 1 "GND" H 7300 1950 60  0000 C CNN
 F 2 "" H 7300 2100 60  0000 C CNN
@@
 RX
 $Comp
-L GND #PWR034
+L GND #PWR033
 U 1 1 549DFFDB
 P 7000 4000
-F 0 "#PWR034" H 7000 3750 60  0001 C CNN
+F 0 "#PWR033" H 7000 3750 60  0001 C CNN
 F 1 "GND" H 7000 3850 60  0000 C CNN
 F 2 "" H 7000 4000 60  0000 C CNN
@@
 $EndComp
 $Comp
-L GND #PWR035
+L GND #PWR034
 U 1 1 549E0E20
 P 9600 3900
-F 0 "#PWR035" H 9600 3650 60  0001 C CNN
+F 0 "#PWR034" H 9600 3650 60  0001 C CNN
 F 1 "GND" H 9600 3750 60  0000 C CNN
 F 2 "" H 9600 3900 60  0000 C CNN
@@
 	9500 3600 9700 3600
 $Comp
-L GND #PWR036
+L GND #PWR035
 U 1 1 549E0F20
 P 8900 4300
-F 0 "#PWR036" H 8900 4050 60  0001 C CNN
+F 0 "#PWR035" H 8900 4050 60  0001 C CNN
 F 1 "GND" H 8900 4150 60  0000 C CNN
 F 2 "" H 8900 4300 60  0000 C CNN
@@
 $EndComp
 $Comp
-L GND #PWR037
+L GND #PWR036
 U 1 1 549E0F34
 P 8200 4300
-F 0 "#PWR037" H 8200 4050 60  0001 C CNN
+F 0 "#PWR036" H 8200 4050 60  0001 C CNN
 F 1 "GND" H 8200 4150 60  0000 C CNN
 F 2 "" H 8200 4300 60  0000 C CNN
@@
 	0    -1   1    0
 $EndComp
+Text Label 2900 1600 0    60   ~ 0
+TxRamp
+Wire Wire Line
+	2900 1600 2800 1600
 $EndSCHEMATC
